File: kicad-files/OpenHardwareHolterMonitor.sch (KiCad schematic (older format))
At the start: 24 parts, among them CON1 Micro_SD_Card, J1 Conn_01x14, P1 Custom_FTDI, Q1 S8050, Q2 S8050, Q3 Q_NMOS_DGS, Q4 Q_NMOS_DGS, U1 ESP-WROOM-32, Y1 32768Hz

Commit message: kicad from git repo
https://git.launchpad.net/kicad
8444b1b6176249060196c22cf0d5027d92f93854

https://git.launchpad.net/kicad-library
bb856328eef2676d859dfa179a6c078922a42274
Parts:
- removed D1: D_Schottky, Diodes_SMD:D_SOD-323_HandSoldering, symbol D_Schottky
- C1, C2: symbol C -> OpenHardwareHolterMonitor-rescue:C
- CON1: symbol Micro_SD_Card -> OpenHardwareHolterMonitor-rescue:Micro_SD_Card
- J1: symbol Conn_01x14 -> OpenHardwareHolterMonitor-rescue:Conn_01x14
- P1: symbol CONN_01X07 -> OpenHardwareHolterMonitor-rescue:CONN_01X07
- Q1, Q2: symbol S8050 -> OpenHardwareHolterMonitor-rescue:S8050
- Q3, Q4: symbol Q_NMOS_DGS -> OpenHardwareHolterMonitor-rescue:Q_NMOS_DGS
- R1, R10, R11, R12, R2, R3, R4, R5, R6, R7, R8, R9: symbol R -> OpenHardwareHolterMonitor-rescue:R
- U1: symbol ESP-WROOM-32 -> esp32:ESP-WROOM-32
- Y1: symbol Crystal -> OpenHardwareHolterMonitor-rescue:Crystal
Changed lines of the file:
@@
-EESchema Schematic File Version 2
-LIBS:OpenHardwareHolterMonitor-rescue
-LIBS:power
-LIBS:device
-LIBS:transistors
-LIBS:conn
-LIBS:linear
-LIBS:regul
-LIBS:74xx
-LIBS:cmos4000
-LIBS:adc-dac
-LIBS:memory
-LIBS:xilinx
-LIBS:microcontrollers
-LIBS:dsp
-LIBS:microchip
-LIBS:analog_switches
-LIBS:motorola
-LIBS:texas
-LIBS:intel
-LIBS:audio
-LIBS:interface
-LIBS:digital-audio
-LIBS:philips
-LIBS:display
-LIBS:cypress
-LIBS:siliconi
-LIBS:opto
-LIBS:atmel
-LIBS:contrib
-LIBS:valves
-LIBS:esp32
-LIBS:ads1299
-LIBS:ads1298
-LIBS:mcp73833
-LIBS:lp5912
-LIBS:rem_3-xxxxs
-LIBS:switches
-LIBS:tps2113a
+EESchema Schematic File Version 4
 LIBS:OpenHardwareHolterMonitor-cache
-EELAYER 25 0
+EELAYER 26 0
 EELAYER END
 $Descr A4 11693 8268
@@
 $EndDescr
 $Comp
-L ESP-WROOM-32 U1
+L esp32:ESP-WROOM-32 U1
 U 1 1 5A22CCAC
 P 2550 2550
@@
 	4200 2200 6150 2200
 $Comp
-L Micro_SD_Card CON1
+L OpenHardwareHolterMonitor-rescue:Micro_SD_Card CON1
 U 1 1 5A2BF6C5
 P 2500 5600
@@
 	1500 4650 1500 6550
 Wire Wire Line
-	1500 6550 1900 6550
+	1500 6550 1650 6550
 Wire Wire Line
 	1900 6550 1900 6400
@@
 Connection ~ 1650 6550
 $Comp
-L GND #PWR01
+L OpenHardwareHolterMonitor-rescue:GND #PWR01
 U 1 1 5A2BFB41
 P 1650 6700
@@
 	900  1900 900  2000
 $Comp
-L GND #PWR02
+L OpenHardwareHolterMonitor-rescue:GND #PWR02
 U 1 1 5A2C02E3
 P 900 2000
@@
 	3800 1900 3800 1500
 $Comp
-L GND #PWR03
+L OpenHardwareHolterMonitor-rescue:GND #PWR03
 U 1 1 5A2C0348
 P 3950 1600
@@
 $EndComp
 $Comp
-L S8050 Q1
+L OpenHardwareHolterMonitor-rescue:S8050 Q1
 U 1 1 5A2C0790
 P 4800 4850
@@
 $EndComp
 $Comp
-L S8050 Q2
+L OpenHardwareHolterMonitor-rescue:S8050 Q2
 U 1 1 5A2C0855
 P 4800 5600
@@
 $EndComp
 $Comp
-L R R5
+L OpenHardwareHolterMonitor-rescue:R R5
 U 1 1 5A2C0A57
 P 4350 4850
@@
 $EndComp
 $Comp
-L R R6
+L OpenHardwareHolterMonitor-rescue:R R6
 U 1 1 5A2C0ACC
 P 4350 5600
@@
 	4500 5600 4600 5600
 Wire Wire Line
-	3900 4850 4200 4850
-Wire Wire Line
-	3900 5600 4200 5600
+	3900 4850 4050 4850
+Wire Wire Line
+	3900 5600 4150 5600
 Wire Wire Line
 	4150 5600 4150 5150
@@
 copied from esp32_core_board_v2 schematic
 $Comp
-L CONN_01X07 P1
+L OpenHardwareHolterMonitor-rescue:CONN_01X07 P1
 U 1 1 5A2C102E
 P 5300 6650
@@
 Text Notes 4200 6550 0    60   ~ 0
 Figure out\nflow control
-Wire Wire Line
-	2100 3700 2100 3700
-$Comp
-L GND #PWR04
+$Comp
+L OpenHardwareHolterMonitor-rescue:GND #PWR04
 U 1 1 5A2C1EF3
 P 2100 3700
@@
 	900  1850 900  1600
 $Comp
-L +3V3 #PWR05
+L OpenHardwareHolterMonitor-rescue:+3V3 #PWR05
 U 1 1 5A2C223B
 P 900 1600
@@
 $EndComp
 $Comp
-L +3V3 #PWR06
+L OpenHardwareHolterMonitor-rescue:+3V3 #PWR06
 U 1 1 5A2C2DBB
 P 5350 2900
@@
 	4600 2900 4600 2300
 $Comp
-L +3V3 #PWR07
+L OpenHardwareHolterMonitor-rescue:+3V3 #PWR07
 U 1 1 5A2C271C
 P 1500 4400
@@
 	5350 3100 6150 3100
 Wire Wire Line
-	5350 3200 6150 3200
+	5350 3200 5900 3200
 Wire Wire Line
 	5350 3200 5350 3250
 $Comp
-L GND #PWR08
+L OpenHardwareHolterMonitor-rescue:GND #PWR08
 U 1 1 5A4136E6
 P 5350 3250
@@
 $EndComp
 Wire Wire Line
-	5350 2900 5350 3100
+	5350 2900 5350 2950
 Wire Wire Line
 	5350 2950 5600 2950
@@
 	3950 1500 3950 1600
 $Comp
-L R R1
+L OpenHardwareHolterMonitor-rescue:R R1
 U 1 1 5A50E09F
 P 4350 2000
@@
 $EndComp
 $Comp
-L R R2
+L OpenHardwareHolterMonitor-rescue:R R2
 U 1 1 5A50E4C0
 P 4350 2700
@@
 $EndComp
 $Comp
-L R R3
+L OpenHardwareHolterMonitor-rescue:R R3
 U 1 1 5A50E54F
 P 4350 2800
@@
 	4500 2000 6150 2000
 $Comp
-L R R4
+L OpenHardwareHolterMonitor-rescue:R R4
 U 1 1 5A50EA46
 P 4350 2900
@@
 F6 "~Bat1charging~" I L 6200 4400 60
 F7 "~Bat2Charging~" I L 6200 4550 60
-F8 "FTDI_V_ISO" I L 6200 4700 60
+F8 "FTDI_VIN" I L 6200 4700 50
 $EndSheet
 Wire Wire Line
@@
 	5700 3800 5700 3700
 $Comp
-L +3V3 #PWR09
+L OpenHardwareHolterMonitor-rescue:+3V3 #PWR09
 U 1 1 5AAE0E01
 P 5700 3700
@@
 	5700 3950 5700 4050
 $Comp
-L GND #PWR010
+L OpenHardwareHolterMonitor-rescue:GND #PWR010
 U 1 1 5AAE0F82
 P 5700 4050
@@
 Enable_vbat_read
 $Comp
-L R R8
+L OpenHardwareHolterMonitor-rescue:R R8
 U 1 1 5AB66BDB
 P 8450 3950
@@
 $EndComp
 $Comp
-L R R9
+L OpenHardwareHolterMonitor-rescue:R R9
 U 1 1 5AB66C92
 P 8450 4400
@@
 $EndComp
 $Comp
-L GND #PWR011
+L OpenHardwareHolterMonitor-rescue:GND #PWR011
 U 1 1 5AB66E2D
 P 8450 5200
@@
 	8450 4550 8450 4600
 Wire Wire Line
-	8450 4100 8450 4250
+	8450 4100 8450 4200
 Wire Wire Line
 	8450 4200 7350 4200
@@
 read_bat_1
 Wire Wire Line
-	7350 4800 8150 4800
+	7350 4800 7900 4800
 Wire Wire Line
 	7350 3750 8450 3750
@@
 	8450 3750 8450 3800
 $Comp
-L Q_NMOS_DGS Q3
+L OpenHardwareHolterMonitor-rescue:Q_NMOS_DGS Q3
 U 1 1 5AB6876E
 P 8350 4800
@@
 $EndComp
 Wire Wire Line
-	8450 5000 8450 5200
+	8450 5000 8450 5150
 Text Label 9100 3750 0    60   ~ 0
 Vbat2
@@
 Enable_vbat_read
 $Comp
-L R R11
+L OpenHardwareHolterMonitor-rescue:R R11
 U 1 1 5AB6D16E
 P 10200 3950
@@
 $EndComp
 $Comp
-L R R12
+L OpenHardwareHolterMonitor-rescue:R R12
 U 1 1 5AB6D174
 P 10200 4400
@@
 $EndComp
 $Comp
-L GND #PWR012
+L OpenHardwareHolterMonitor-rescue:GND #PWR012
 U 1 1 5AB6D17A
 P 10200 5200
@@
 	10200 4550 10200 4600
 Wire Wire Line
-	10200 4100 10200 4250
+	10200 4100 10200 4200
 Wire Wire Line
 	10200 4200 9100 4200
@@
 read_bat_2
 Wire Wire Line
-	9100 4800 9900 4800
+	9100 4800 9650 4800
 Wire Wire Line
 	9100 3750 10200 3750
@@
 	10200 3750 10200 3800
 $Comp
-L Q_NMOS_DGS Q4
+L OpenHardwareHolterMonitor-rescue:Q_NMOS_DGS Q4
 U 1 1 5AB6D189
 P 10100 4800
@@
 $EndComp
 Wire Wire Line
-	10200 5000 10200 5200
-$Comp
-L R R10
+	10200 5000 10200 5150
+$Comp
+L OpenHardwareHolterMonitor-rescue:R R10
 U 1 1 5AB6D672
 P 9650 5000
@@
 Connection ~ 10200 5150
 $Comp
-L R R7
+L OpenHardwareHolterMonitor-rescue:R R7
 U 1 1 5AB6DED9
 P 7900 5000
@@
 RTC_N
 $Comp
-L Crystal Y1
+L OpenHardwareHolterMonitor-rescue:Crystal Y1
 U 1 1 5AB80CB4
 P 8250 2300
@@
 	8400 2300 8550 2300
 $Comp
-L C C1
+L OpenHardwareHolterMonitor-rescue:C C1
 U 1 1 5AB811F5
 P 7950 2750
@@
 $EndComp
 $Comp
-L C C2
+L OpenHardwareHolterMonitor-rescue:C C2
 U 1 1 5AB81307
 P 8550 2750
@@
 $EndComp
 Wire Wire Line
-	7950 2000 7950 2600
-Wire Wire Line
-	8550 2000 8550 2600
+	7950 2000 7950 2300
+Wire Wire Line
+	8550 2000 8550 2300
 Connection ~ 7950 2300
 Connection ~ 8550 2300
@@
 	8550 2900 8550 3000
 $Comp
-L GND #PWR013
+L OpenHardwareHolterMonitor-rescue:GND #PWR013
 U 1 1 5AB819C3
 P 7950 3000
@@
 $EndComp
 $Comp
-L GND #PWR014
+L OpenHardwareHolterMonitor-rescue:GND #PWR014
 U 1 1 5AB81ABB
 P 8550 3000
@@
 	9600 2100 9600 2150
 $Comp
-L GND #PWR015
+L OpenHardwareHolterMonitor-rescue:GND #PWR015
 U 1 1 5AB8DBEB
 P 9600 2150
@@
 	9600 2050 9600 1850
 $Comp
-L +3V3 #PWR016
+L OpenHardwareHolterMonitor-rescue:+3V3 #PWR016
 U 1 1 5AB8E0DB
 P 9600 1850
@@
 $EndComp
 Wire Wire Line
-	6200 4700 6150 4700
-Wire Wire Line
-	5850 4700 5500 4700
-Text Label 5500 4700 0    60   ~ 0
+	6200 4700 5850 4700
+Text Label 5850 4700 0    60   ~ 0
 FTDI_V
-$Comp
-L D_Schottky D1
-U 1 1 5AB94F8B
-P 6000 4700
-F 0 "D1" H 6000 4800 50  0000 C CNN
-F 1 "D_Schottky" H 6000 4600 50  0000 C CNN
-F 2 "Diodes_SMD:D_SOD-323_HandSoldering" H 6000 4700 50  0001 C CNN
-F 3 "" H 6000 4700 50  0000 C CNN
-	1    6000 4700
-	-1   0    0    1
-$EndComp
 Wire Wire Line
 	5100 6350 4800 6350
@@
 IO13
 $Comp
-L Conn_01x14 J1
+L OpenHardwareHolterMonitor-rescue:Conn_01x14 J1
 U 1 1 5B164661
 P 10400 2700
@@
 Text Notes 4400 7100 0    60   ~ 0
 TODO - Custom FTDI?
+Wire Wire Line
+	1650 6550 1900 6550
+Wire Wire Line
+	4150 5600 4200 5600
+Wire Wire Line
+	4050 4850 4200 4850
+Wire Wire Line
+	5350 2950 5350 3100
+Wire Wire Line
+	5900 3200 6150 3200
+Wire Wire Line
+	8450 4200 8450 4250
+Wire Wire Line
+	10200 4200 10200 4250
+Wire Wire Line
+	10200 5150 10200 5200
+Wire Wire Line
+	8450 5150 8450 5200
+Wire Wire Line
+	7900 4800 8150 4800
+Wire Wire Line
+	9650 4800 9900 4800
+Wire Wire Line
+	7950 2300 7950 2600
+Wire Wire Line
+	8550 2300 8550 2600
 $EndSCHEMATC
