File: kicad-files/OpenHardwareHolterMonitor.sch (KiCad schematic (older format))
At the start: 23 parts, among them CON1 Micro_SD_Card, J1 Conn_01x14, P1 Custom_FTDI, Q1 S8050, Q2 S8050, Q3 Q_NMOS_DGS, Q4 Q_NMOS_DGS, U1 ESP-WROOM-32, Y1 32768Hz

Commit message: more footprint usage
Parts:
- U1: footprint (none) -> ESP-WROOM-32:MODULE_ESP-WROOM-32
Changed lines of the file:
@@
 F 0 "U1" H 2550 2550 60  0000 C CNN
 F 1 "ESP-WROOM-32" H 2550 2650 60  0000 C CNN
-F 2 "" H 2550 2550 60  0001 C CNN
+F 2 "ESP-WROOM-32:MODULE_ESP-WROOM-32" H 2550 2550 60  0001 C CNN
 F 3 "" H 2550 2550 60  0001 C CNN
 	1    2550 2550

Commit message: finish footprints
Parts:
- Y1: footprint (none) -> crystals:K161
Changed lines of the file:
@@
 F 0 "Y1" H 8250 2450 50  0000 C CNN
 F 1 "32768Hz" H 8250 2150 50  0000 C CNN
-F 2 "" H 8250 2300 50  0001 C CNN
+F 2 "crystals:K161" H 8250 2300 50  0001 C CNN
 F 3 "" H 8250 2300 50  0000 C CNN
 	1    8250 2300

Commit message: checkpoint; non-isolated layout
Connections:
- net labels added: SD_CD, SD_CLK, SD_DAT0, SD_DAT1, SD_DAT2, SD_VSS, START_OUT, ~CS~, ~DRDY~_IN, ~PWDN~_OUT, ~RESET~_OUT
- net labels removed: CS
Changed lines of the file:
@@
 CLK
 Text Label 4100 2800 2    60   ~ 0
-CS
+~CS~
 Text Label 4100 2000 2    60   ~ 0
 MOSI
@@
 Wire Wire Line
 	8550 2300 8550 2600
+Text Label 3800 2100 0    50   ~ 0
+~PWDN~_OUT
+Text Label 3750 2400 0    50   ~ 0
+~RESET~_OUT
+Text Label 3800 3000 0    50   ~ 0
+~DRDY~_IN
+Text Label 3750 2900 0    50   ~ 0
+START_OUT
+Text Label 2100 4550 1    50   ~ 0
+SD_DAT1
+Text Label 2200 4550 1    50   ~ 0
+SD_DAT0
+Text Label 1500 4950 1    50   ~ 0
+SD_VSS
+Text Label 2600 4350 1    50   ~ 0
+SD_CLK
+Text Label 2800 4650 1    50   ~ 0
+SD_DAT2
+Text Label 2700 4650 1    50   ~ 0
+SD_CD
 $EndSCHEMATC

Commit message: add battery reversal protection to schematic
Connections:
- net labels added: Enable_Charging
- net labels removed: IO26
- wire segments 174 -> 175
Other:
- moved on the sheet: Q1, Q2, R5, R6
Changed lines of the file:
@@
 L OpenHardwareHolterMonitor-rescue:S8050 Q1
 U 1 1 5A2C0790
-P 4800 4850
-F 0 "Q1" H 5000 4925 50  0000 L CNN
-F 1 "S8050" H 5000 4850 50  0000 L CNN
-F 2 "TO_SOT_Packages_SMD:SOT-23_Handsoldering" H 5000 4775 50  0000 L CIN
-F 3 "" H 4800 4850 50  0000 L CNN
-	1    4800 4850
+P 4700 5050
+F 0 "Q1" H 4900 5125 50  0000 L CNN
+F 1 "S8050" H 4900 5050 50  0000 L CNN
+F 2 "TO_SOT_Packages_SMD:SOT-23_Handsoldering" H 4900 4975 50  0000 L CIN
+F 3 "" H 4700 5050 50  0000 L CNN
+	1    4700 5050
 	1    0    0    -1
 $EndComp
@@
 L OpenHardwareHolterMonitor-rescue:S8050 Q2
 U 1 1 5A2C0855
-P 4800 5600
-F 0 "Q2" H 5000 5675 50  0000 L CNN
-F 1 "S8050" H 5000 5600 50  0000 L CNN
-F 2 "TO_SOT_Packages_SMD:SOT-23_Handsoldering" H 5000 5525 50  0000 L CIN
-F 3 "" H 4800 5600 50  0000 L CNN
-	1    4800 5600
+P 4700 5800
+F 0 "Q2" H 4900 5875 50  0000 L CNN
+F 1 "S8050" H 4900 5800 50  0000 L CNN
+F 2 "TO_SOT_Packages_SMD:SOT-23_Handsoldering" H 4900 5725 50  0000 L CIN
+F 3 "" H 4700 5800 50  0000 L CNN
+	1    4700 5800
 	1    0    0    1
 $EndComp
@@
 L OpenHardwareHolterMonitor-rescue:R R5
 U 1 1 5A2C0A57
-P 4350 4850
-F 0 "R5" V 4430 4850 50  0000 C CNN
-F 1 "12K" V 4350 4850 50  0000 C CNN
-F 2 "Resistors_SMD:R_0603_HandSoldering" V 4280 4850 50  0001 C CNN
-F 3 "" H 4350 4850 50  0000 C CNN
-	1    4350 4850
+P 4250 5050
+F 0 "R5" V 4330 5050 50  0000 C CNN
+F 1 "12K" V 4250 5050 50  0000 C CNN
+F 2 "Resistors_SMD:R_0603_HandSoldering" V 4180 5050 50  0001 C CNN
+F 3 "" H 4250 5050 50  0000 C CNN
+	1    4250 5050
 	0    1    1    0
 $EndComp
@@
 L OpenHardwareHolterMonitor-rescue:R R6
 U 1 1 5A2C0ACC
-P 4350 5600
-F 0 "R6" V 4430 5600 50  0000 C CNN
-F 1 "12K" V 4350 5600 50  0000 C CNN
-F 2 "Resistors_SMD:R_0603_HandSoldering" V 4280 5600 50  0001 C CNN
-F 3 "" H 4350 5600 50  0000 C CNN
-	1    4350 5600
+P 4250 5800
+F 0 "R6" V 4330 5800 50  0000 C CNN
+F 1 "12K" V 4250 5800 50  0000 C CNN
+F 2 "Resistors_SMD:R_0603_HandSoldering" V 4180 5800 50  0001 C CNN
+F 3 "" H 4250 5800 50  0000 C CNN
+	1    4250 5800
 	0    1    1    0
 $EndComp
 Wire Wire Line
-	4500 4850 4600 4850
-Wire Wire Line
-	4500 5600 4600 5600
-Wire Wire Line
-	3900 4850 4050 4850
-Wire Wire Line
-	3900 5600 4150 5600
-Wire Wire Line
-	4150 5600 4150 5150
-Wire Wire Line
-	4150 5150 4900 5150
-Wire Wire Line
-	4900 5150 4900 5050
-Connection ~ 4150 5600
-Wire Wire Line
-	4050 4850 4050 5250
-Wire Wire Line
-	4050 5250 4900 5250
-Wire Wire Line
-	4900 5250 4900 5400
-Connection ~ 4050 4850
-Text Label 3900 4850 0    60   ~ 0
+	4400 5050 4500 5050
+Wire Wire Line
+	4400 5800 4500 5800
+Wire Wire Line
+	3800 5050 3950 5050
+Wire Wire Line
+	3800 5800 4050 5800
+Wire Wire Line
+	4050 5800 4050 5350
+Wire Wire Line
+	4050 5350 4800 5350
+Wire Wire Line
+	4800 5350 4800 5250
+Connection ~ 4050 5800
+Wire Wire Line
+	3950 5050 3950 5450
+Wire Wire Line
+	3950 5450 4800 5450
+Wire Wire Line
+	4800 5450 4800 5600
+Connection ~ 3950 5050
+Text Label 3800 5050 0    60   ~ 0
 DTR
-Text Label 3900 5600 0    60   ~ 0
+Text Label 3800 5800 0    60   ~ 0
 RTS
 Wire Wire Line
-	4900 4650 4900 4600
-Wire Wire Line
-	4900 4600 5250 4600
-Wire Wire Line
-	4900 5800 4900 5900
-Wire Wire Line
-	4900 5900 5250 5900
-Text Label 5250 5900 2    60   ~ 0
+	4800 4850 4800 4800
+Wire Wire Line
+	4800 4800 5150 4800
+Wire Wire Line
+	4800 6000 4800 6100
+Wire Wire Line
+	4800 6100 5150 6100
+Text Label 5150 6100 2    60   ~ 0
 IO0
-Text Label 5250 4600 2    60   ~ 0
+Text Label 5150 4800 2    60   ~ 0
 EN
-Text Notes 4000 4600 0    30   ~ 0
+Text Notes 3900 4800 0    30   ~ 0
 copied from esp32_core_board_v2 schematic
 $Comp
@@
 F7 "~Bat2Charging~" I L 6200 4550 60
 F8 "FTDI_VIN" I L 6200 4700 50
+F9 "Enable_Charging" I L 6200 4850 50
 $EndSheet
 Wire Wire Line
@@
 Text Label 1100 2300 0    60   ~ 0
 IO39
-Text Label 1100 2900 0    60   ~ 0
-IO26
 Text Label 1100 3000 0    60   ~ 0
 IO27
@@
 IO12
 Wire Wire Line
-	1400 2900 1100 2900
-Wire Wire Line
 	1400 3000 1100 3000
 Wire Wire Line
@@
 	1400 3200 1100 3200
 Text Label 9900 2900 0    60   ~ 0
-IO26
-Text Label 9900 3000 0    60   ~ 0
 IO27
 Text Label 9900 2700 0    60   ~ 0
@@
 	10200 2900 9900 2900
 Wire Wire Line
+	10200 2700 9900 2700
+Wire Wire Line
+	10200 2500 9900 2500
+Wire Wire Line
 	10200 3000 9900 3000
-Wire Wire Line
-	10200 2700 9900 2700
-Wire Wire Line
-	10200 2500 9900 2500
+Text Label 9900 3000 0    60   ~ 0
+IO36
 Wire Wire Line
 	10200 3100 9900 3100
 Text Label 9900 3100 0    60   ~ 0
-IO36
-Wire Wire Line
-	10200 3200 9900 3200
-Text Label 9900 3200 0    60   ~ 0
 IO39
 Text Label 2900 4000 1    60   ~ 0
@@
 	1650 6550 1900 6550
 Wire Wire Line
-	4150 5600 4200 5600
-Wire Wire Line
-	4050 4850 4200 4850
+	4050 5800 4100 5800
+Wire Wire Line
+	3950 5050 4100 5050
 Wire Wire Line
 	5350 2950 5350 3100
@@
 Text Label 2700 4650 1    50   ~ 0
 SD_CD
+Wire Wire Line
+	6200 4850 5500 4850
+Text Label 5500 4850 0    50   ~ 0
+Enable_Charging
+Wire Wire Line
+	550  2900 1400 2900
+Text Label 550  2900 0    50   ~ 0
+Enable_Charging
+Text Label 9550 3200 0    50   ~ 0
+Enable_Charging
+Wire Wire Line
+	9550 3200 10200 3200
 $EndSCHEMATC

Commit message: board layout checkpoint
Parts:
- removed J1: Conn_01x14, Pin_Headers:Pin_Header_Straight_1x14_Pitch2.54mm, symbol OpenHardwareHolterMonitor-rescue:Conn_01x14
- added J1: Conn_02x06_Odd_Even, Pin_Headers:Pin_Header_Straight_2x06_Pitch1.27mm, symbol Connector:Conn_02x06_Odd_Even
- added TP1, TP2, TP3: Test_Point, Measurement_Points:Measurement_Point_Square-SMD-Pad_Small, symbol Connector:Test_Point
Connections:
- wire segments 175 -> 177
Changed lines of the file:
@@
 Wire Wire Line
 	1400 3200 1100 3200
-Text Label 9900 2900 0    60   ~ 0
+Text Label 11000 2500 2    60   ~ 0
 IO27
-Text Label 9900 2700 0    60   ~ 0
+Text Label 11000 2400 2    60   ~ 0
 IO14
-Text Label 9900 2500 0    60   ~ 0
+Text Label 11000 2300 2    60   ~ 0
 IO12
 Wire Wire Line
-	10200 2900 9900 2900
-Wire Wire Line
-	10200 2700 9900 2700
-Wire Wire Line
-	10200 2500 9900 2500
-Wire Wire Line
-	10200 3000 9900 3000
-Text Label 9900 3000 0    60   ~ 0
+	11000 2500 10700 2500
+Wire Wire Line
+	11000 2400 10700 2400
+Wire Wire Line
+	11000 2300 10700 2300
+Wire Wire Line
+	9900 2600 10200 2600
+Text Label 9900 2600 0    60   ~ 0
 IO36
 Wire Wire Line
-	10200 3100 9900 3100
-Text Label 9900 3100 0    60   ~ 0
+	10700 2600 11000 2600
+Text Label 11000 2600 2    60   ~ 0
 IO39
 Text Label 2900 4000 1    60   ~ 0
@@
 Wire Wire Line
 	2900 3700 2900 4000
-Text Label 9900 2800 0    60   ~ 0
+Text Label 9900 2500 0    60   ~ 0
 IO15
 Wire Wire Line
-	10200 2800 9900 2800
+	9900 2500 10200 2500
 Text Label 4000 3100 2    60   ~ 0
 IO4
 Wire Wire Line
 	3700 3100 4000 3100
-Text Label 9900 2400 0    60   ~ 0
+Text Label 9900 2300 0    60   ~ 0
 IO4
 Wire Wire Line
-	10200 2400 9900 2400
-Wire Wire Line
-	10200 2200 9900 2200
-Wire Wire Line
-	10200 2100 9600 2100
+	10200 2300 9900 2300
 Wire Wire Line
 	9600 2100 9600 2150
@@
 $EndComp
 Wire Wire Line
-	9900 2200 9900 2050
-Wire Wire Line
 	9900 2050 9600 2050
 Wire Wire Line
@@
 DTR
 Wire Wire Line
-	10200 3300 9900 3300
-Wire Wire Line
-	10200 3400 9900 3400
-Text Label 9900 3300 0    60   ~ 0
+	10200 5800 9900 5800
+Wire Wire Line
+	10200 6000 9900 6000
+Text Label 9900 5800 0    60   ~ 0
 Vbat1
-Text Label 9900 3400 0    60   ~ 0
+Text Label 9900 6000 0    60   ~ 0
 Vbat2
 Wire Wire Line
@@
 IO13
 Wire Wire Line
-	10200 2600 9900 2600
-Text Label 9900 2600 0    60   ~ 0
+	9900 2400 10200 2400
+Text Label 9900 2400 0    60   ~ 0
 IO13
-$Comp
-L OpenHardwareHolterMonitor-rescue:Conn_01x14 J1
-U 1 1 5B164661
-P 10400 2700
-F 0 "J1" H 10400 3400 50  0000 C CNN
-F 1 "Conn_01x14" H 10400 1900 50  0000 C CNN
-F 2 "Pin_Headers:Pin_Header_Straight_1x14_Pitch2.54mm" H 10400 2700 50  0001 C CNN
-F 3 "" H 10400 2700 50  0001 C CNN
-	1    10400 2700
-	1    0    0    -1
-$EndComp
-Wire Wire Line
-	10200 2300 9900 2300
-Text Label 9900 2300 0    60   ~ 0
+Wire Wire Line
+	10700 2200 11000 2200
+Text Label 11000 2200 2    60   ~ 0
 IO2
 NoConn ~ 4800 6750
@@
 Text Label 550  2900 0    50   ~ 0
 Enable_Charging
-Text Label 9550 3200 0    50   ~ 0
+Text Label 9550 5600 0    50   ~ 0
 Enable_Charging
 Wire Wire Line
-	9550 3200 10200 3200
+	9550 5600 10200 5600
+$Comp
+L Connector:Test_Point TP1
+U 1 1 5C99AAF0
+P 10200 5600
+F 0 "TP1" V 10154 5788 50  0000 L CNN
+F 1 "Test_Point" V 10245 5788 50  0000 L CNN
+F 2 "Measurement_Points:Measurement_Point_Square-SMD-Pad_Small" H 10400 5600 50  0001 C CNN
+F 3 "~" H 10400 5600 50  0001 C CNN
+	1    10200 5600
+	0    1    1    0
+$EndComp
+$Comp
+L Connector:Test_Point TP2
+U 1 1 5C99ABBF
+P 10200 5800
+F 0 "TP2" V 10154 5988 50  0000 L CNN
+F 1 "Test_Point" V 10245 5988 50  0000 L CNN
+F 2 "Measurement_Points:Measurement_Point_Square-SMD-Pad_Small" H 10400 5800 50  0001 C CNN
+F 3 "~" H 10400 5800 50  0001 C CNN
+	1    10200 5800
+	0    1    1    0
+$EndComp
+$Comp
+L Connector:Test_Point TP3
+U 1 1 5C99AC98
+P 10200 6000
+F 0 "TP3" V 10154 6188 50  0000 L CNN
+F 1 "Test_Point" V 10245 6188 50  0000 L CNN
+F 2 "Measurement_Points:Measurement_Point_Square-SMD-Pad_Small" H 10400 6000 50  0001 C CNN
+F 3 "~" H 10400 6000 50  0001 C CNN
+	1    10200 6000
+	0    1    1    0
+$EndComp
+$Comp
+L Connector:Conn_02x06_Odd_Even J1
+U 1 1 5CAE7D82
+P 10400 2300
+F 0 "J1" H 10450 2717 50  0000 C CNN
+F 1 "Conn_02x06_Odd_Even" H 10450 2626 50  0000 C CNN
+F 2 "Pin_Headers:Pin_Header_Straight_2x06_Pitch1.27mm" H 10400 2300 50  0001 C CNN
+F 3 "~" H 10400 2300 50  0001 C CNN
+	1    10400 2300
+	1    0    0    -1
+$EndComp
+Wire Wire Line
+	11100 2100 11100 2150
+$Comp
+L OpenHardwareHolterMonitor-rescue:GND #PWR0102
+U 1 1 5CAE7EA9
+P 11100 2150
+F 0 "#PWR0102" H 11100 1900 50  0001 C CNN
+F 1 "GND" H 11100 2000 50  0000 C CNN
+F 2 "" H 11100 2150 50  0000 C CNN
+F 3 "" H 11100 2150 50  0000 C CNN
+	1    11100 2150
+	1    0    0    -1
+$EndComp
+Wire Wire Line
+	10700 2100 11100 2100
+Wire Wire Line
+	9600 2100 10200 2100
+Wire Wire Line
+	9900 2050 9900 2200
+Wire Wire Line
+	9900 2200 10200 2200
 $EndSCHEMATC

Commit message: esp-wroom footprint update
Parts:
- U1: footprint ESP-WROOM-32:MODULE_ESP-WROOM-32 -> esp-wroom-32:MODULE_ESP-WROOM-32
Changed lines of the file:
@@
 F 0 "U1" H 2550 2550 60  0000 C CNN
 F 1 "ESP-WROOM-32" H 2550 2650 60  0000 C CNN
-F 2 "ESP-WROOM-32:MODULE_ESP-WROOM-32" H 2550 2550 60  0001 C CNN
+F 2 "esp-wroom-32:MODULE_ESP-WROOM-32" H 2550 2550 60  0001 C CNN
 F 3 "" H 2550 2550 60  0001 C CNN
 	1    2550 2550

Commit message: align physical items with schematic
Parts:
- added MH_NE1, MH_NW1, MH_SE1, MH_SW1: Mounting_Hole, Mounting_Holes:MountingHole_2.2mm_M2_ISO7380, symbol Mechanical:Mounting_Hole
- Y1: manufacturer-pn (none) -> FK161EIHM0.032768
Connections:
- net GND: now also U1.1.1 (GND_PAD)
Changed lines of the file:
@@
 	1500 4600 1500 4400
 Wire Wire Line
-	1400 1900 900  1900
+	1400 1900 1350 1900
 Wire Wire Line
 	900  1900 900  2000
@@
 F 2 "crystals:K161" H 8250 2300 50  0001 C CNN
 F 3 "" H 8250 2300 50  0000 C CNN
+F 4 "FK161EIHM0.032768" H 8250 2300 50  0000 C CNN "manufacturer-pn"
 	1    8250 2300
 	1    0    0    -1
@@
 Wire Wire Line
 	9900 2200 10200 2200
+Wire Wire Line
+	1400 1800 1350 1800
+Wire Wire Line
+	1350 1800 1350 1900
+Connection ~ 1350 1900
+Wire Wire Line
+	1350 1900 900  1900
+$Comp
+L Mechanical:Mounting_Hole MH_NW1
+U 1 1 5C1F5248
+P 850 7150
+F 0 "MH_NW1" H 950 7196 50  0000 L CNN
+F 1 "Mounting_Hole" H 950 7105 50  0000 L CNN
+F 2 "Mounting_Holes:MountingHole_2.2mm_M2_ISO7380" H 850 7150 50  0001 C CNN
+F 3 "" H 850 7150 50  0001 C CNN
+	1    850  7150
+	1    0    0    -1
+$EndComp
+$Comp
+L Mechanical:Mounting_Hole MH_SW1
+U 1 1 5C1F5695
+P 850 7450
+F 0 "MH_SW1" H 950 7496 50  0000 L CNN
+F 1 "Mounting_Hole" H 950 7405 50  0000 L CNN
+F 2 "Mounting_Holes:MountingHole_2.2mm_M2_ISO7380" H 850 7450 50  0001 C CNN
+F 3 "" H 850 7450 50  0001 C CNN
+	1    850  7450
+	1    0    0    -1
+$EndComp
+$Comp
+L Mechanical:Mounting_Hole MH_NE1
+U 1 1 5C1F5739
+P 2000 7150
+F 0 "MH_NE1" H 2100 7196 50  0000 L CNN
+F 1 "Mounting_Hole" H 2100 7105 50  0000 L CNN
+F 2 "Mounting_Holes:MountingHole_2.2mm_M2_ISO7380" H 2000 7150 50  0001 C CNN
+F 3 "" H 2000 7150 50  0001 C CNN
+	1    2000 7150
+	1    0    0    -1
+$EndComp
+$Comp
+L Mechanical:Mounting_Hole MH_SE1
+U 1 1 5C1F57DC
+P 2000 7450
+F 0 "MH_SE1" H 2100 7496 50  0000 L CNN
+F 1 "Mounting_Hole" H 2100 7405 50  0000 L CNN
+F 2 "Mounting_Holes:MountingHole_2.2mm_M2_ISO7380" H 2000 7450 50  0001 C CNN
+F 3 "" H 2000 7450 50  0001 C CNN
+	1    2000 7450
+	1    0    0    -1
+$EndComp
 $EndSCHEMATC

Commit message: add the first few part numbers
Parts:
- C1, C2: manufacturer-pn (none) -> C0603C120J5GAC
Other:
- note removed: "FK161"
Changed lines of the file:
@@
 U 1 1 5AB80CB4
 P 8250 2300
-F 0 "Y1" H 8250 2450 50  0000 C CNN
-F 1 "32768Hz" H 8250 2150 50  0000 C CNN
+F 0 "Y1" V 8250 2300 50  0000 C CNN
+F 1 "32768Hz" H 8250 2450 50  0000 C CNN
 F 2 "crystals:K161" H 8250 2300 50  0001 C CNN
 F 3 "" H 8250 2300 50  0000 C CNN
-F 4 "FK161EIHM0.032768" H 8250 2300 50  0000 C CNN "manufacturer-pn"
+F 4 "FK161EIHM0.032768" H 8250 2150 50  0000 C CNN "manufacturer-pn"
 	1    8250 2300
 	1    0    0    -1
@@
 F 2 "Capacitors_SMD:C_0603_HandSoldering" H 7988 2600 50  0001 C CNN
 F 3 "" H 7950 2750 50  0000 C CNN
+F 4 "C0603C120J5GAC" H 0   0   50  0001 C CNN "manufacturer-pn"
 	1    7950 2750
 	1    0    0    -1
@@
 F 2 "Capacitors_SMD:C_0603_HandSoldering" H 8588 2600 50  0001 C CNN
 F 3 "" H 8550 2750 50  0000 C CNN
+F 4 "C0603C120J5GAC" H 0   0   50  0001 C CNN "manufacturer-pn"
 	1    8550 2750
 	1    0    0    -1
@@
 Text Label 8550 2000 0    60   ~ 0
 RTC_N
-Text Notes 8300 2400 1    30   ~ 0
-FK161
 Wire Wire Line
 	1400 2200 1100 2200
