File: kicad-files/ads1298.sch (KiCad schematic (older format))
At the start: 46 parts

Commit message: multiplex power-in
Other:
- note added: "TODO: Consider external clock"
Changed lines of the file:
@@
 LIBS:rem_3-xxxxs
 LIBS:switches
+LIBS:tps2113a
 LIBS:OpenHardwareHolterMonitor-cache
 EELAYER 25 0
@@
 chest
 Connection ~ 7500 3100
+Text Notes 4800 6350 0    60   ~ 0
+TODO: Consider external clock
 $EndSCHEMATC

Commit message: fix rules-check issues
Parts:
- added J10, J11, J12, J13, J4, J5, J6, J7, J8, J9: Conn_01x01, symbol Conn_01x01
- gave numbers to parts that had none: 46
Connections:
- net IN1_8N: now also J6.1 (Pin_1)
- net IN2P: now also J7.1 (Pin_1)
- net IN3P: now also J8.1 (Pin_1)
- net IN4P: now also J9.1 (Pin_1)
- net IN5P: now also J10.1 (Pin_1)
- net IN6P: now also J11.1 (Pin_1)
- net IN7P: now also J12.1 (Pin_1)
- net IN8P: now also J13.1 (Pin_1)
- net INP1: now also J5.1 (Pin_1)
- net RLDOUT: now also J4.1 (Pin_1)

Commit message: assign some footprints
Parts:
- C10, C11, C13, C14, C15, C16, C17, C18, C19, C20, C21, C22, C23, C24, C25, C26, C27, C28, C29, C3, C30, C31, C32, C33, C4, C5, C6, C7, C9: footprint (none) -> Capacitors_SMD:C_0603_HandSoldering
- C12, C8: footprint (none) -> Capacitors_SMD:C_0805_HandSoldering
- R13, R14, R15, R16: footprint (none) -> Resistors_SMD:R_0603_HandSoldering
- R17, R18, R19, R20, R21, R22, R23, R24, R25, R26: footprint (none) -> Resistors_ThroughHole:R_Axial_Power_L20.0mm_W6.4mm_P25.40mm
- renumbered J12 to J10, J13 to J11, J4 to J2, J5 to J3, J6 to J4, J7 to J5, J8 to J6, J9 to J7, J10 to J8, J11 to J9
Other:
- note added: "C8 Could be tantilum for vibration resistance"

Commit message: kicad from git repo
https://git.launchpad.net/kicad
8444b1b6176249060196c22cf0d5027d92f93854

https://git.launchpad.net/kicad-library
bb856328eef2676d859dfa179a6c078922a42274
Parts:
- C10, C11, C12, C13, C14, C15, C16, C17, C18, C19, C20, C21, C22, C23, C24, C25, C26, C27, C28, C29, C3, C30, C31, C32, C33, C4, C5, C6, C7, C8, C9: symbol C -> OpenHardwareHolterMonitor-rescue:C
- J10, J11, J2, J3, J4, J5, J6, J7, J8, J9: symbol Conn_01x01 -> OpenHardwareHolterMonitor-rescue:Conn_01x01
- R13, R14, R15, R16, R17, R18, R19, R20, R21, R22, R23, R24, R25, R26: symbol R -> OpenHardwareHolterMonitor-rescue:R
- U2: symbol ADS1298 -> ads1298:ADS1298

Commit message: add some footprints
Parts:
- U2: footprint (none) -> Housings_QFP:LQFP-64_10x10mm_Pitch0.5mm
Changed lines of the file:
@@
 F 0 "U2" H 5350 3550 60  0000 C CNN
 F 1 "ADS1298" H 5350 3950 60  0000 C CNN
-F 2 "" H 5350 3750 60  0001 C CNN
+F 2 "Housings_QFP:LQFP-64_10x10mm_Pitch0.5mm" H 5350 3750 60  0001 C CNN
 F 3 "" H 5350 3750 60  0001 C CNN
 	1    5350 3750
