File: kicad-files/power.sch (KiCad schematic (older format))
At the start: 45 parts, among them J2 USB_OTG, J3 USB_C_Receptacle, SW1 SW_Push_Open, U3 MCP73833, U4 MCP73833, U5 TPS2113A, U6 LP5912, U7 REM_3-xxxxS

Commit message: assign some footprints
Parts:
- removed R36: 10, symbol R
- added C35, C37: 330uF, Capacitors_Tantalum_SMD:CP_Tantalum_Case-E_EIA-7260-38_Hand, symbol CP
- BT1, BT2: footprint (none) -> Connectors_JST:JST_PH_S2B-PH-SM4-TB_02x2.00mm_Angled
- C34: value 1mF -> 330uF; footprint (none) -> Capacitors_Tantalum_SMD:CP_Tantalum_Case-E_EIA-7260-38_Hand
- C36: renamed from C35; footprint (none) -> Capacitors_SMD:C_0603_HandSoldering
- C38: renamed from C37; footprint (none) -> Capacitors_SMD:C_0603_HandSoldering
- C39: renamed from C36; footprint (none) -> Capacitors_SMD:C_0805_HandSoldering
- C40: renamed from C39; footprint (none) -> Capacitors_SMD:C_0805_HandSoldering
- C41: renamed from C38; footprint (none) -> Capacitors_SMD:C_0805_HandSoldering
- C42: renamed from C40; footprint (none) -> Capacitors_SMD:C_0805_HandSoldering
- D2, D3, D4, D5, D6, D7: footprint (none) -> Diodes_SMD:D_SOD-323_HandSoldering
- D8: footprint (none) -> TO_SOT_Packages_SMD:TO-277A
- D9: footprint (none) -> LEDs:LED_0603_HandSoldering
- F1, F2: footprint (none) -> Resistors_SMD:R_1812_HandSoldering
- J12: renamed from J2; footprint (none) -> Connectors_USB:USB_Micro-B_Wuerth-629105150521_CircularHoles
- J13: renamed from J3; footprint (none) -> Connectors_USB:USB_C_Receptacle_Amphenol_12401610E4-2A_CircularHoles
- R27, R28: value R -> 100k; footprint (none) -> Resistors_SMD:R_0603_HandSoldering
- R29, R30, R31, R32, R33, R34, R35: footprint (none) -> Resistors_SMD:R_0603_HandSoldering
- R36: renamed from R37; value R -> NI; footprint (none) -> Resistors_SMD:R_0603_HandSoldering
Connections:
- wire segments 175 -> 176
- no-connect marks 20 -> 21
Other:
- note added: "REM3-0505 Data sheet recommends\n1000uF through-hole Nippon Chemi-con KY series\nwe replaced with 3 SMD tantalums\n"
- note removed: "Nippon Chemi-con KY series"
- moved on the sheet: C39, C41, FL1

Commit message: kicad from git repo
https://git.launchpad.net/kicad
8444b1b6176249060196c22cf0d5027d92f93854

https://git.launchpad.net/kicad-library
bb856328eef2676d859dfa179a6c078922a42274
Parts:
- removed SW1: SW_Push_Open, symbol SW_Push_Open
- added D1, D10: D_Schottky, Diodes_SMD:D_SOD-323_HandSoldering, symbol OpenHardwareHolterMonitor-rescue:D_Schottky
- added SW1: SW_SPST, symbol Switch:SW_SPST
- BT1, BT2: symbol Battery_Cell -> OpenHardwareHolterMonitor-rescue:Battery_Cell
- C34, C35, C37: symbol CP -> OpenHardwareHolterMonitor-rescue:CP
- C36, C38, C39, C40, C41, C42: symbol C -> OpenHardwareHolterMonitor-rescue:C
- D2, D3, D6, D7: symbol D_Schottky -> OpenHardwareHolterMonitor-rescue:D_Schottky
- D4, D5: symbol D_Zener -> OpenHardwareHolterMonitor-rescue:D_Zener
- D8: symbol D_Schottky_AAK -> OpenHardwareHolterMonitor-rescue:D_Schottky_AAK
- D9: symbol LED -> OpenHardwareHolterMonitor-rescue:LED
- F1, F2: symbol Polyfuse -> OpenHardwareHolterMonitor-rescue:Polyfuse
- FL1: symbol EMI_Filter_LL -> OpenHardwareHolterMonitor-rescue:EMI_Filter_LL
- J12: symbol USB_OTG -> OpenHardwareHolterMonitor-rescue:USB_OTG
- J13: symbol USB_C_Receptacle -> OpenHardwareHolterMonitor-rescue:USB_C_Receptacle
- R27, R28, R29, R30, R31, R32, R33, R34, R35, R36: symbol R -> OpenHardwareHolterMonitor-rescue:R
- TH1, TH2: symbol Thermistor_NTC -> OpenHardwareHolterMonitor-rescue:Thermistor_NTC
- TP1, TP2, TP3, TP4: symbol TEST -> OpenHardwareHolterMonitor-rescue:TEST
- U3, U4: symbol MCP73833 -> mcp73833:MCP73833
- U5: symbol TPS2113A -> tps2113a:TPS2113A
- U6: symbol LP5912 -> lp5912:LP5912
- U7: symbol REM_3-xxxxS -> rem_3-xxxxs:REM_3-xxxxS
Connections:
- net labels added: FTDI_VIN
- net labels removed: FTDI_V_ISO, VBAT1, VBAT2
- wire segments 176 -> 244

Commit message: add some footprints
Parts:
- TH1, TH2: footprint (none) -> Capacitors_ThroughHole:CP_Radial_D4.0mm_P1.50mm
- TP1, TP2, TP3, TP4: footprint (none) -> Pin_Headers:Pin_Header_Straight_1x01_Pitch2.54mm
- U3, U4: footprint (none) -> Housings_SSOP:MSOP-10_3x3mm_Pitch0.5mm
- U5: footprint (none) -> Housings_SSOP:TSSOP-8_4.4x3mm_Pitch0.65mm
Other:
- note added: "ALPS SSSS810701"
- note added: "Keystone Electronics 1043"
Changed lines of the file:
@@
 F 0 "U4" H 3000 4250 60  0000 C CNN
 F 1 "MCP73833" H 3000 4150 60  0000 C CNN
-F 2 "" H 3000 4200 60  0001 C CNN
+F 2 "Housings_SSOP:MSOP-10_3x3mm_Pitch0.5mm" H 3000 4200 60  0001 C CNN
 F 3 "" H 3000 4200 60  0001 C CNN
 	1    3000 4200
@@
 F 0 "TP2" H 950 5050 50  0000 C BNN
 F 1 "TEST" H 950 5000 50  0000 C CNN
-F 2 "" H 950 4750 50  0001 C CNN
+F 2 "Pin_Headers:Pin_Header_Straight_1x01_Pitch2.54mm" H 950 4750 50  0001 C CNN
 F 3 "" H 950 4750 50  0000 C CNN
 	1    950  4750
@@
 F 0 "TP4" H 4300 5050 50  0000 C BNN
 F 1 "TEST" H 4300 5000 50  0000 C CNN
-F 2 "" H 4300 4750 50  0001 C CNN
+F 2 "Pin_Headers:Pin_Header_Straight_1x01_Pitch2.54mm" H 4300 4750 50  0001 C CNN
 F 3 "" H 4300 4750 50  0000 C CNN
 	1    4300 4750
@@
 F 0 "TH2" V 4675 4800 50  0000 C CNN
 F 1 "Thermistor_NTC" V 4975 4800 50  0000 C CNN
-F 2 "" H 4850 4850 50  0001 C CNN
+F 2 "Capacitors_ThroughHole:CP_Radial_D4.0mm_P1.50mm" H 4850 4850 50  0001 C CNN
 F 3 "" H 4850 4850 50  0001 C CNN
 	1    4850 4800
@@
 F 0 "U3" H 2950 6350 60  0000 C CNN
 F 1 "MCP73833" H 2950 6250 60  0000 C CNN
-F 2 "" H 2950 6300 60  0001 C CNN
+F 2 "Housings_SSOP:MSOP-10_3x3mm_Pitch0.5mm" H 2950 6300 60  0001 C CNN
 F 3 "" H 2950 6300 60  0001 C CNN
 	1    2950 6300
@@
 F 0 "TP1" H 900 7150 50  0000 C BNN
 F 1 "TEST" H 900 7100 50  0000 C CNN
-F 2 "" H 900 6850 50  0001 C CNN
+F 2 "Pin_Headers:Pin_Header_Straight_1x01_Pitch2.54mm" H 900 6850 50  0001 C CNN
 F 3 "" H 900 6850 50  0000 C CNN
 	1    900  6850
@@
 F 0 "TP3" H 4250 7150 50  0000 C BNN
 F 1 "TEST" H 4250 7100 50  0000 C CNN
-F 2 "" H 4250 6850 50  0001 C CNN
+F 2 "Pin_Headers:Pin_Header_Straight_1x01_Pitch2.54mm" H 4250 6850 50  0001 C CNN
 F 3 "" H 4250 6850 50  0000 C CNN
 	1    4250 6850
@@
 F 0 "TH1" V 4625 6900 50  0000 C CNN
 F 1 "Thermistor_NTC" V 4925 6900 50  0000 C CNN
-F 2 "" H 4800 6950 50  0001 C CNN
+F 2 "Capacitors_ThroughHole:CP_Radial_D4.0mm_P1.50mm" H 4800 6950 50  0001 C CNN
 F 3 "" H 4800 6950 50  0001 C CNN
 	1    4800 6900
@@
 F 0 "U5" H 5950 1450 60  0000 C CNN
 F 1 "TPS2113A" H 5950 1350 60  0000 C CNN
-F 2 "" H 5950 1350 60  0001 C CNN
+F 2 "Housings_SSOP:TSSOP-8_4.4x3mm_Pitch0.65mm" H 5950 1350 60  0001 C CNN
 F 3 "" H 5950 1350 60  0001 C CNN
 	1    5950 1350
@@
 	8500 2850 8550 2850
 Connection ~ 8500 2750
+Text Notes 7600 3950 0    30   ~ 0
+ALPS SSSS810701
+Text Notes 4650 6450 0    30   ~ 0
+Keystone  Electronics 1043
+Text Notes 4700 4350 0    30   ~ 0
+Keystone  Electronics 1043
 $EndSCHEMATC

Commit message: more footprints
Parts:
- removed SW1: SW_SPST, symbol Switch:SW_SPST
- added SW1: SW_SPDT, Alps:ALPS_SSSS810701, symbol Switch:SW_SPDT
- FL1: footprint (none) -> CMS1:CMS1
- J12: footprint Connectors_USB:USB_Micro-B_Wuerth-629105150521_CircularHoles -> PlasticsOne:PlasticsOne_41828
Connections:
- net labels removed: GND_ISO
- wire segments 244 -> 252
- no-connect marks 21 -> 22
Other:
- note added: "ALPS SSSS811101"
- note removed: "ALPS SSSS810701"
- moved on the sheet: C40, C42
Changed lines of the file:
@@
 	-1   0    0    1
 $EndComp
-Text Label 1150 4400 0    60   ~ 0
-GND_ISO
 Text Label 4900 4000 2    60   ~ 0
 Vbat1
@@
 	1    0    0    -1
 $EndComp
-Text Label 4650 4500 0    60   ~ 0
-GND_ISO
 $Comp
 L OpenHardwareHolterMonitor-rescue:D_Schottky D7
@@
 	-1   0    0    -1
 $EndComp
-Text Label 6800 4000 0    60   ~ 0
+Text Label 6600 4100 0    60   ~ 0
 REGULATOR_IN
 Text Label 6450 4000 2    60   ~ 0
 REGULATOR_IN
-Text Label 6800 4100 0    60   ~ 0
-GND_ISO
 Text Label 10700 4000 2    60   ~ 0
 3v3
-Text Label 9850 4100 2    60   ~ 0
-GND_ISO
-Text Label 8850 4650 2    60   ~ 0
-GND_ISO
 $Comp
 L OpenHardwareHolterMonitor-rescue:TEST TP2
@@
 	1    0    0    -1
 $EndComp
-Text Label 4400 5200 0    60   ~ 0
-GND_ISO
 $Comp
 L OpenHardwareHolterMonitor-rescue:R R32
@@
 	0    -1   -1   0
 $EndComp
-Text Notes 4000 5400 0    30   ~ 0
+Text Notes 4000 5450 0    30   ~ 0
 MCP Datasheet typical: approx 5C-40C\nWith series resistor of 276 Ohm and parallel resistor of 149751 Ohm\n would give range of approx: 0C-45C
 $Comp
 L OpenHardwareHolterMonitor-rescue:C C40
 U 1 1 5AAD2225
-P 8150 4450
+P 7900 4300
 AR Path="/5AAD2225" Ref="C40"  Part="1"
 AR Path="/5A6D4EDD/5AAD2225" Ref="C40"  Part="1"
-F 0 "C40" H 8175 4550 50  0000 L CNN
-F 1 "10uF" H 8175 4350 50  0000 L CNN
-F 2 "Capacitors_SMD:C_0805_HandSoldering" H 8188 4300 50  0001 C CNN
-F 3 "" H 8150 4450 50  0000 C CNN
-	1    8150 4450
+F 0 "C40" H 7925 4400 50  0000 L CNN
+F 1 "10uF" H 7925 4200 50  0000 L CNN
+F 2 "Capacitors_SMD:C_0805_HandSoldering" H 7938 4150 50  0001 C CNN
+F 3 "" H 7900 4300 50  0000 C CNN
+	1    7900 4300
 	1    0    0    -1
 $EndComp
@@
 L OpenHardwareHolterMonitor-rescue:C C42
 U 1 1 5AAD236E
-P 10400 4450
+P 10400 4250
 AR Path="/5AAD236E" Ref="C42"  Part="1"
 AR Path="/5A6D4EDD/5AAD236E" Ref="C42"  Part="1"
-F 0 "C42" H 10425 4550 50  0000 L CNN
-F 1 "10uF" H 10425 4350 50  0000 L CNN
-F 2 "Capacitors_SMD:C_0805_HandSoldering" H 10438 4300 50  0001 C CNN
-F 3 "" H 10400 4450 50  0000 C CNN
-	1    10400 4450
+F 0 "C42" H 10425 4350 50  0000 L CNN
+F 1 "10uF" H 10425 4150 50  0000 L CNN
+F 2 "Capacitors_SMD:C_0805_HandSoldering" H 10438 4100 50  0001 C CNN
+F 3 "" H 10400 4250 50  0000 C CNN
+	1    10400 4250
 	1    0    0    -1
 $EndComp
@@
 	-1   0    0    1
 $EndComp
-Text Label 1100 6500 0    60   ~ 0
-GND_ISO
 Text Label 4850 6100 2    60   ~ 0
 Vbat2
@@
 	1    0    0    -1
 $EndComp
-Text Label 4600 6600 0    60   ~ 0
-GND_ISO
 $Comp
 L OpenHardwareHolterMonitor-rescue:D_Schottky D6
@@
 	1    0    0    -1
 $EndComp
-Text Label 4350 7300 0    60   ~ 0
-GND_ISO
 $Comp
 L OpenHardwareHolterMonitor-rescue:R R31
@@
 	0    -1   -1   0
 $EndComp
-Text Notes 3950 7500 0    30   ~ 0
+Text Notes 3950 7550 0    30   ~ 0
 MCP Datasheet typical: approx 5C-40C\nWith series resistor of 276 Ohm and parallel resistor of 149751 Ohm\n would give range of approx: 0C-45C
 Text Label 5000 800  2    60   ~ 0
 Bat2_Stat1
 Text Label 1550 800  2    60   ~ 0
-GND_ISO
+GND
 Text Label 3350 650  2    60   ~ 0
 Vbat1
@@
 F 0 "FL1" H 7800 2975 50  0000 C CNN
 F 1 "131uH" H 7800 2625 50  0000 C CNN
-F 2 "" V 7800 2840 50  0001 C CNN
+F 2 "CMS1:CMS1" V 7800 2840 50  0001 C CNN
 F 3 "" V 7800 2840 50  0000 C CNN
 	1    7800 2800
@@
 V_ISO
 Text Label 10750 2650 2    60   ~ 0
-GND_ISO
+GND
 Text HLabel 5800 650  0    60   Input ~ 0
 FTDI_VIN
@@
 F 0 "J12" H 1600 1950 50  0000 L CNN
 F 1 "USB_OTG" H 1600 1850 50  0000 L CNN
-F 2 "Connectors_USB:USB_Micro-B_Wuerth-629105150521_CircularHoles" H 1950 1450 50  0001 C CNN
+F 2 "PlasticsOne:PlasticsOne_41828" H 1950 1450 50  0001 C CNN
 F 3 "" H 1950 1450 50  0001 C CNN
 	1    1800 1500
@@
 Connection ~ 2050 4000
 Wire Wire Line
-	2200 4400 1150 4400
-Wire Wire Line
 	3800 4000 4000 4000
 Wire Wire Line
@@
 	4650 4000 4650 4050
 Wire Wire Line
-	4650 4350 4650 4500
+	4650 4350 4650 4400
 Connection ~ 4650 4000
 Wire Wire Line
-	8000 4000 8050 4000
-Wire Wire Line
 	5500 4000 6450 4000
 Wire Wire Line
-	8250 4100 6800 4100
-Wire Wire Line
 	9450 4000 10400 4000
 Wire Wire Line
-	9450 4100 9850 4100
-Wire Wire Line
 	8850 4500 8850 4650
 Wire Wire Line
-	2200 4300 2100 4300
-Wire Wire Line
-	2100 4300 2100 4800
-Wire Wire Line
-	2100 4800 950  4800
+	2200 4300 2050 4300
+Wire Wire Line
+	2050 4300 2050 4800
+Wire Wire Line
+	2050 4800 950  4800
 Wire Wire Line
 	950  4800 950  4750
@@
 Connection ~ 4400 5050
 Wire Wire Line
-	8150 4300 8150 4000
-Connection ~ 8150 4000
-Wire Wire Line
-	8150 4600 8150 4650
-Wire Wire Line
-	8150 4650 8850 4650
-Wire Wire Line
-	10400 4300 10400 4000
+	10400 4100 10400 4000
 Connection ~ 10400 4000
 Wire Wire Line
-	10400 4650 10400 4600
+	10400 4650 10400 4400
 Connection ~ 8850 4650
 Wire Wire Line
@@
 Connection ~ 2000 6100
 Wire Wire Line
-	2150 6500 1100 6500
-Wire Wire Line
 	3750 6100 3950 6100
 Wire Wire Line
@@
 	4600 6100 4600 6150
 Wire Wire Line
-	4600 6450 4600 6600
+	4600 6450 4600 6500
 Connection ~ 4600 6100
 Wire Wire Line
 	5450 6100 6400 6100
 Wire Wire Line
-	2150 6400 2050 6400
-Wire Wire Line
-	2050 6400 2050 6900
-Wire Wire Line
-	2050 6900 900  6900
+	2150 6400 2000 6400
+Wire Wire Line
+	2000 6400 2000 6900
+Wire Wire Line
+	2000 6900 900  6900
 Wire Wire Line
 	900  6900 900  6850
@@
 	10250 2650 10750 2650
 Wire Wire Line
-	6800 4000 7500 4000
-Wire Wire Line
 	6300 650  7100 650
 Wire Wire Line
@@
 	8050 3900 8050 4000
 Connection ~ 8050 4000
-Wire Wire Line
-	7500 4000 7500 4200
-Wire Wire Line
-	7500 4200 8250 4200
-Connection ~ 7500 4000
 Wire Wire Line
 	1900 3900 1900 4000
@@
 	4400 4200 4550 4200
 Wire Wire Line
-	4400 5050 4400 5200
+	4400 5050 4400 5100
 Wire Wire Line
 	4400 5050 4000 5050
 Wire Wire Line
-	8150 4000 8250 4000
-Wire Wire Line
 	10400 4000 10700 4000
 Wire Wire Line
-	8850 4650 10400 4650
+	8850 4650 9550 4650
 Wire Wire Line
 	2000 6100 2150 6100
@@
 	4350 6300 4500 6300
 Wire Wire Line
-	4350 7150 4350 7300
+	4350 7150 4350 7200
 Wire Wire Line
 	4350 7150 3950 7150
@@
 Wire Wire Line
 	8100 3150 8100 3450
-Wire Wire Line
-	8050 4000 8150 4000
-Wire Wire Line
-	7500 4000 7600 4000
 Wire Wire Line
 	1900 4000 2050 4000
@@
 Text Label 8900 3500 0    50   ~ 0
 V_ISO
-$Comp
-L Switch:SW_SPST SW1
-U 1 1 5B21EA3A
-P 7800 4000
-F 0 "SW1" H 7800 4235 50  0000 C CNN
-F 1 "SW_SPST" H 7800 4144 50  0000 C CNN
-F 2 "" H 7800 4000 50  0001 C CNN
-F 3 "" H 7800 4000 50  0001 C CNN
-	1    7800 4000
-	1    0    0    -1
-$EndComp
 Text Label 7100 650  2    60   ~ 0
 REGULATOR_IN
@@
 	8500 2850 8550 2850
 Connection ~ 8500 2750
-Text Notes 7600 3950 0    30   ~ 0
-ALPS SSSS810701
+Text Notes 7450 4150 0    30   ~ 0
+ALPS SSSS811101
 Text Notes 4650 6450 0    30   ~ 0
 Keystone  Electronics 1043
 Text Notes 4700 4350 0    30   ~ 0
 Keystone  Electronics 1043
+$Comp
+L Switch:SW_SPDT SW1
+U 1 1 5B269F35
+P 7450 4100
+F 0 "SW1" H 7450 4385 50  0000 C CNN
+F 1 "SW_SPDT" H 7450 4294 50  0000 C CNN
+F 2 "Alps:ALPS_SSSS810701" H 7450 4100 50  0001 C CNN
+F 3 "" H 7450 4100 50  0001 C CNN
+	1    7450 4100
+	1    0    0    -1
+$EndComp
+Wire Wire Line
+	6600 4100 7250 4100
+NoConn ~ 7650 4200
+$Comp
+L power:GND #PWR?
+U 1 1 5B41E505
+P 10700 4850
+F 0 "#PWR?" H 10700 4600 50  0001 C CNN
+F 1 "GND" H 10705 4677 50  0000 C CNN
+F 2 "" H 10700 4850 50  0001 C CNN
+F 3 "" H 10700 4850 50  0001 C CNN
+	1    10700 4850
+	1    0    0    -1
+$EndComp
+Wire Wire Line
+	10700 4650 10700 4850
+Wire Wire Line
+	8050 4000 8150 4000
+Wire Wire Line
+	8250 4100 8200 4100
+Wire Wire Line
+	8200 4100 8200 4650
+Connection ~ 8200 4650
+Wire Wire Line
+	8200 4650 8850 4650
+Wire Wire Line
+	7650 4000 7900 4000
+Wire Wire Line
+	8250 4200 8150 4200
+Wire Wire Line
+	8150 4200 8150 4000
+Connection ~ 8150 4000
+Wire Wire Line
+	8150 4000 8250 4000
+Wire Wire Line
+	7900 4000 7900 4150
+Connection ~ 7900 4000
+Wire Wire Line
+	7900 4000 8050 4000
+Wire Wire Line
+	7900 4450 7900 4650
+Wire Wire Line
+	9450 4100 9550 4100
+Wire Wire Line
+	9550 4100 9550 4650
+Connection ~ 9550 4650
+Wire Wire Line
+	9550 4650 10400 4650
+Wire Wire Line
+	10400 4650 10700 4650
+Connection ~ 10400 4650
+Wire Wire Line
+	7900 4650 8200 4650
+$Comp
+L power:GND #PWR?
+U 1 1 5B61EC7F
+P 4650 4400
+F 0 "#PWR?" H 4650 4150 50  0001 C CNN
+F 1 "GND" H 4655 4227 50  0000 C CNN
+F 2 "" H 4650 4400 50  0001 C CNN
+F 3 "" H 4650 4400 50  0001 C CNN
+	1    4650 4400
+	1    0    0    -1
+$EndComp
+$Comp
+L power:GND #PWR?
+U 1 1 5B62E702
+P 4400 5100
+F 0 "#PWR?" H 4400 4850 50  0001 C CNN
+F 1 "GND" H 4405 4927 50  0000 C CNN
+F 2 "" H 4400 5100 50  0001 C CNN
+F 3 "" H 4400 5100 50  0001 C CNN
+	1    4400 5100
+	1    0    0    -1
+$EndComp
+$Comp
+L power:GND #PWR?
+U 1 1 5B64DDF2
+P 4350 7200
+F 0 "#PWR?" H 4350 6950 50  0001 C CNN
+F 1 "GND" H 4355 7027 50  0000 C CNN
+F 2 "" H 4350 7200 50  0001 C CNN
+F 3 "" H 4350 7200 50  0001 C CNN
+	1    4350 7200
+	1    0    0    -1
+$EndComp
+Wire Wire Line
+	2150 6500 2100 6500
+Wire Wire Line
+	2100 6500 2100 6600
+$Comp
+L power:GND #PWR?
+U 1 1 5B68C8D1
+P 2100 6600
+F 0 "#PWR?" H 2100 6350 50  0001 C CNN
+F 1 "GND" H 2105 6427 50  0000 C CNN
+F 2 "" H 2100 6600 50  0001 C CNN
+F 3 "" H 2100 6600 50  0001 C CNN
+	1    2100 6600
+	1    0    0    -1
+$EndComp
+Wire Wire Line
+	2200 4400 2150 4400
+Wire Wire Line
+	2150 4400 2150 4500
+$Comp
+L power:GND #PWR?
+U 1 1 5B6EB6A1
+P 2150 4500
+F 0 "#PWR?" H 2150 4250 50  0001 C CNN
+F 1 "GND" H 2155 4327 50  0000 C CNN
+F 2 "" H 2150 4500 50  0001 C CNN
+F 3 "" H 2150 4500 50  0001 C CNN
+	1    2150 4500
+	1    0    0    -1
+$EndComp
+$Comp
+L power:GND #PWR?
+U 1 1 5B6FB9BD
+P 4600 6500
+F 0 "#PWR?" H 4600 6250 50  0001 C CNN
+F 1 "GND" H 4605 6327 50  0000 C CNN
+F 2 "" H 4600 6500 50  0001 C CNN
+F 3 "" H 4600 6500 50  0001 C CNN
+	1    4600 6500
+	1    0    0    -1
+$EndComp
 $EndSCHEMATC

Commit message: more footprint usage
Parts:
- U6: footprint (none) -> WSON:WSON-6_2x2mm_Pitch0.65mm
Changed lines of the file:
@@
 F 0 "U6" H 8850 4250 60  0000 C CNN
 F 1 "LP5912" H 8850 4150 60  0000 C CNN
-F 2 "" H 8850 4100 60  0001 C CNN
+F 2 "WSON:WSON-6_2x2mm_Pitch0.65mm" H 8850 4100 60  0001 C CNN
 F 3 "" H 8850 4100 60  0001 C CNN
 	1    8850 4100
@@
 NoConn ~ 7650 4200
 $Comp
-L power:GND #PWR?
+L power:GND #PWR0101
 U 1 1 5B41E505
 P 10700 4850
-F 0 "#PWR?" H 10700 4600 50  0001 C CNN
+F 0 "#PWR0101" H 10700 4600 50  0001 C CNN
 F 1 "GND" H 10705 4677 50  0000 C CNN
 F 2 "" H 10700 4850 50  0001 C CNN
@@
 	7900 4650 8200 4650
 $Comp
-L power:GND #PWR?
+L power:GND #PWR0102
 U 1 1 5B61EC7F
 P 4650 4400
-F 0 "#PWR?" H 4650 4150 50  0001 C CNN
+F 0 "#PWR0102" H 4650 4150 50  0001 C CNN
 F 1 "GND" H 4655 4227 50  0000 C CNN
 F 2 "" H 4650 4400 50  0001 C CNN
@@
 $EndComp
 $Comp
-L power:GND #PWR?
+L power:GND #PWR0103
 U 1 1 5B62E702
 P 4400 5100
-F 0 "#PWR?" H 4400 4850 50  0001 C CNN
+F 0 "#PWR0103" H 4400 4850 50  0001 C CNN
 F 1 "GND" H 4405 4927 50  0000 C CNN
 F 2 "" H 4400 5100 50  0001 C CNN
@@
 $EndComp
 $Comp
-L power:GND #PWR?
+L power:GND #PWR0104
 U 1 1 5B64DDF2
 P 4350 7200
-F 0 "#PWR?" H 4350 6950 50  0001 C CNN
+F 0 "#PWR0104" H 4350 6950 50  0001 C CNN
 F 1 "GND" H 4355 7027 50  0000 C CNN
 F 2 "" H 4350 7200 50  0001 C CNN
@@
 	2100 6500 2100 6600
 $Comp
-L power:GND #PWR?
+L power:GND #PWR0105
 U 1 1 5B68C8D1
 P 2100 6600
-F 0 "#PWR?" H 2100 6350 50  0001 C CNN
+F 0 "#PWR0105" H 2100 6350 50  0001 C CNN
 F 1 "GND" H 2105 6427 50  0000 C CNN
 F 2 "" H 2100 6600 50  0001 C CNN
@@
 	2150 4400 2150 4500
 $Comp
-L power:GND #PWR?
+L power:GND #PWR0106
 U 1 1 5B6EB6A1
 P 2150 4500
-F 0 "#PWR?" H 2150 4250 50  0001 C CNN
+F 0 "#PWR0106" H 2150 4250 50  0001 C CNN
 F 1 "GND" H 2155 4327 50  0000 C CNN
 F 2 "" H 2150 4500 50  0001 C CNN
@@
 $EndComp
 $Comp
-L power:GND #PWR?
+L power:GND #PWR0107
 U 1 1 5B6FB9BD
 P 4600 6500
-F 0 "#PWR?" H 4600 6250 50  0001 C CNN
+F 0 "#PWR0107" H 4600 6250 50  0001 C CNN
 F 1 "GND" H 4605 6327 50  0000 C CNN
 F 2 "" H 4600 6500 50  0001 C CNN

Commit message: finish footprints
Parts:
- U7: footprint (none) -> isolators:REM3
Changed lines of the file:
@@
 F 0 "U7" H 9400 2800 60  0000 C CNN
 F 1 "REM_3-xxxxS" H 9400 2650 60  0000 C CNN
-F 2 "" H 9400 2800 60  0001 C CNN
+F 2 "isolators:REM3" H 9400 2800 60  0001 C CNN
 F 3 "" H 9400 2800 60  0001 C CNN
 	1    9400 2800

Commit message: checkpoint initial pcb file
Parts:
- J12: footprint PlasticsOne:PlasticsOne_41828 -> Connectors_USB:USB_Micro-B_Wuerth-629105150521_CircularHoles
Changed lines of the file:
@@
 F 0 "J12" H 1600 1950 50  0000 L CNN
 F 1 "USB_OTG" H 1600 1850 50  0000 L CNN
-F 2 "PlasticsOne:PlasticsOne_41828" H 1950 1450 50  0001 C CNN
+F 2 "Connectors_USB:USB_Micro-B_Wuerth-629105150521_CircularHoles" H 1950 1450 50  0001 C CNN
 F 3 "" H 1950 1450 50  0001 C CNN
 	1    1800 1500

Commit message: checkpoint 3 pcb file
Parts:
- BT1, BT2: footprint Connectors_JST:JST_PH_S2B-PH-SM4-TB_02x2.00mm_Angled -> keystone1043:Keystone1043
Changed lines of the file:
@@
 F 0 "BT2" H 4750 4350 50  0000 L CNN
 F 1 "Battery_Cell" H 4750 4250 50  0000 L CNN
-F 2 "Connectors_JST:JST_PH_S2B-PH-SM4-TB_02x2.00mm_Angled" V 4650 4310 50  0001 C CNN
+F 2 "keystone1043:Keystone1043" V 4650 4310 50  0001 C CNN
 F 3 "" V 4650 4310 50  0000 C CNN
 	1    4650 4250
@@
 F 0 "BT1" H 4700 6450 50  0000 L CNN
 F 1 "Battery_Cell" H 4700 6350 50  0000 L CNN
-F 2 "Connectors_JST:JST_PH_S2B-PH-SM4-TB_02x2.00mm_Angled" V 4600 6410 50  0001 C CNN
+F 2 "keystone1043:Keystone1043" V 4600 6410 50  0001 C CNN
 F 3 "" V 4600 6410 50  0000 C CNN
 	1    4600 6350
