File: kicad-files/power.sch (KiCad schematic (older format))
At the start: 65 parts, among them J12 USB_OTG, J13 USB_C_Receptacle, Q10 Q_PMOS_DGS, Q5 Q_NMOS_DGS, Q6 Q_NMOS_DGS, Q7 Q_PMOS_DGS, Q8 Q_PMOS_DGS, Q9 Q_PMOS_DGS, SW1 SW_SPDT, U3 MCP73833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

Commit message: replace switch and rework pcb
Parts:
- added Q11: Q_PMOS_DGS, TO_SOT_Packages_SMD:SOT-23_Handsoldering, symbol OpenHardwareHolterMonitor-rescue:Q_PMOS_DGS-device
- Q10, Q7, Q8, Q9: ManufacturerName (none) -> Diodes Incorporated; manufacturer-pn (none) -> DMG2305UX
- SW1: footprint Alps:ALPS_SSSS810701 -> Buttons_Switches_SMD:SW_SPDT_CK-JS102011SAQN; symbol OpenHardwareHolterMonitor-rescue:ALPS_SSSS810701-ALPS -> Switch:SW_SPDT; ManufacturerName TODO: Digikey does not stock -> C&K; manufacturer-pn SSSS810701 -> JS102011SAQN
Connections:
- net GND: now also SW1.3 (C); no longer SW1.SHIELD (Shield)
- net REGULATOR_IN: now also C40.1, U6.4 (EN), U6.6 (IN), Q11.1 (D); no longer D1.1 (K), D10.1 (K), D12.1 (K), D6.1 (K), SW1.2 (B)
- new net: Q11.2 (G), SW1.2 (B)
- new net SWITCH_IN: D1.1 (K), D10.1 (K), D12.1 (K), D6.1 (K), Q11.3 (S), SW1.1 (A)
- no-connect marks 22 -> 21
Other:
- note removed: "ALPS SSSS811101"
Changed lines of the file:
@@
 	-1   0    0    -1
 $EndComp
-Text Label 7000 5500 0    60   ~ 0
-REGULATOR_IN
+Text Label 6850 4850 0    60   ~ 0
+SWITCH_IN
 Text Label 11100 5400 2    60   ~ 0
 3v3
@@
 $EndComp
 Text Label 7850 5900 2    60   ~ 0
-REGULATOR_IN
+SWITCH_IN
 $Comp
 L OpenHardwareHolterMonitor-rescue:R R29
@@
 $EndComp
 Text Label 11100 4350 2    60   ~ 0
-REGULATOR_IN
+SWITCH_IN
 Wire Wire Line
 	10150 4350 11100 4350
@@
 V_ISO
 Text Label 11150 1800 2    60   ~ 0
-REGULATOR_IN
+SWITCH_IN
 $Comp
 L OpenHardwareHolterMonitor-rescue:D_Schottky D?
@@
 	8500 2850 8550 2850
 Connection ~ 8500 2750
-Text Notes 7850 5550 0    30   ~ 0
-ALPS SSSS811101
 Text Notes 6300 7400 0    30   ~ 0
 Keystone  Electronics 1043
 $Comp
-L OpenHardwareHolterMonitor-rescue:ALPS_SSSS810701-ALPS SW1
+L Switch:SW_SPDT SW1
 U 1 1 5B269F35
-P 7850 5500
+P 7400 5250
 AR Path="/5B269F35" Ref="SW1"  Part="1"
 AR Path="/5A6D4EDD/5B269F35" Ref="SW1"  Part="1"
-F 0 "SW1" H 7850 5785 50  0000 C CNN
-F 1 "SW_SPDT" H 7850 5694 50  0000 C CNN
-F 2 "Alps:ALPS_SSSS810701" H 7850 5500 50  0001 C CNN
-F 3 "" H 7850 5500 50  0001 C CNN
-F 4 "SSSS810701" H 7850 5500 50  0000 C CNN "manufacturer-pn"
-F 5 "TODO: Digikey does not stock" H 0   0   50  0001 C CNN "ManufacturerName"
-	1    7850 5500
-	1    0    0    -1
-$EndComp
-Wire Wire Line
-	7000 5500 7650 5500
-NoConn ~ 8050 5600
+F 0 "SW1" H 7400 5535 50  0000 C CNN
+F 1 "SW_SPDT" H 7400 5444 50  0000 C CNN
+F 2 "Buttons_Switches_SMD:SW_SPDT_CK-JS102011SAQN" H 7400 5250 50  0001 C CNN
+F 3 "" H 7400 5250 50  0001 C CNN
+F 4 "JS102011SAQN" H 7400 5250 50  0001 C CNN "manufacturer-pn"
+F 5 "C&K" H -450 -250 50  0001 C CNN "ManufacturerName"
+	1    7400 5250
+	-1   0    0    -1
+$EndComp
 $Comp
 L power:GND #PWR0101
@@
 F 2 "TO_SOT_Packages_SMD:SOT-23_Handsoldering" H 5250 6300 50  0001 C CNN
 F 3 "" H 5050 6200 50  0001 C CNN
+F 4 "Diodes Incorporated" H 0   0   50  0001 C CNN "ManufacturerName"
+F 5 "DMG2305UX" H 0   0   50  0001 C CNN "manufacturer-pn"
 	1    5050 6200
 	-1   0    0    1
@@
 F 2 "TO_SOT_Packages_SMD:SOT-23_Handsoldering" H 5850 6300 50  0001 C CNN
 F 3 "" H 5650 6200 50  0001 C CNN
+F 4 "Diodes Incorporated" H 0   0   50  0001 C CNN "ManufacturerName"
+F 5 "DMG2305UX" H 0   0   50  0001 C CNN "manufacturer-pn"
 	1    5650 6200
 	1    0    0    1
@@
 	-1   0    0    1
 $EndComp
-Text Label 7850 4100 2    60   ~ 0
+Text Label 8050 5400 0    60   ~ 0
 REGULATOR_IN
 $Comp
@@
 F 2 "TO_SOT_Packages_SMD:SOT-23_Handsoldering" H 5250 4500 50  0001 C CNN
 F 3 "" H 5050 4400 50  0001 C CNN
+F 4 "Diodes Incorporated" H 0   0   50  0001 C CNN "ManufacturerName"
+F 5 "DMG2305UX" H 0   0   50  0001 C CNN "manufacturer-pn"
 	1    5050 4400
 	-1   0    0    1
@@
 F 2 "TO_SOT_Packages_SMD:SOT-23_Handsoldering" H 5850 4500 50  0001 C CNN
 F 3 "" H 5650 4400 50  0001 C CNN
+F 4 "Diodes Incorporated" H 0   0   50  0001 C CNN "ManufacturerName"
+F 5 "DMG2305UX" H 0   0   50  0001 C CNN "manufacturer-pn"
 	1    5650 4400
 	1    0    0    1
@@
 Text Notes 2150 7450 0    30   ~ 0
 Consider thermal pad and SMD
-Wire Wire Line
-	7750 5700 6550 5700
-Wire Wire Line
-	6550 5700 6550 5600
-Wire Wire Line
-	6550 5600 6250 5600
+$Comp
+L OpenHardwareHolterMonitor-rescue:Q_PMOS_DGS-device Q11
+U 1 1 5C48123F
+P 7700 4950
+F 0 "Q11" V 7906 4904 50  0000 L CNN
+F 1 "Q_PMOS_DGS" V 7550 4950 50  0000 L CNN
+F 2 "TO_SOT_Packages_SMD:SOT-23_Handsoldering" H 7900 5050 50  0001 C CNN
+F 3 "" H 7700 4950 50  0001 C CNN
+F 4 "Diodes Incorporated" H 2650 550 50  0001 C CNN "ManufacturerName"
+F 5 "DMG2305UX" H 2650 550 50  0001 C CNN "manufacturer-pn"
+	1    7700 4950
+	0    1    -1   0
+$EndComp
+Wire Wire Line
+	7900 4850 8050 4850
+Wire Wire Line
+	8050 4850 8050 5400
+Wire Wire Line
+	7200 5150 7000 5150
+$Comp
+L power:GND #PWR0103
+U 1 1 5C6276AF
+P 7150 5500
+F 0 "#PWR0103" H 7150 5250 50  0001 C CNN
+F 1 "GND" H 7155 5327 50  0000 C CNN
+F 2 "" H 7150 5500 50  0001 C CNN
+F 3 "" H 7150 5500 50  0001 C CNN
+	1    7150 5500
+	1    0    0    -1
+$EndComp
+Wire Wire Line
+	6850 4850 7000 4850
+Wire Wire Line
+	7000 5150 7000 4850
+Connection ~ 7000 4850
+Wire Wire Line
+	7000 4850 7500 4850
+Wire Wire Line
+	7600 5250 7700 5250
+Wire Wire Line
+	7700 5250 7700 5150
+Text Label 7850 4100 2    50   ~ 0
+SWITCH_IN
+Wire Wire Line
+	7200 5350 7150 5350
+Wire Wire Line
+	7150 5350 7150 5500
 $EndSCHEMATC

Commit message: more parts of the BOM
Parts:
- D11, D7: ManufacturerName (none) -> Inolux; manufacturer-pn (none) -> IN-S63BTA
- D4, D5: footprint Diodes_SMD:D_SOD-323_HandSoldering -> Diodes_SMD:D_SMB_Handsoldering; ManufacturerName (none) -> Micro Commercial Components (MCC); manufacturer-pn (none) -> SMBJ5339B-TP
- D8: manufacturer-pn V10P45S-M3/86A -> TPS2113A
- D9: ManufacturerName (none) -> Lite-On Inc.; manufacturer-pn (none) -> LTST-C191KGKT
- F1, F2: manufacturer-pn 2920L050DR -> F8132CT-ND
Changed lines of the file:
@@
 F 3 "" H 6200 2750 50  0000 C CNN
 F 4 "Vishay" H 0   0   50  0001 C CNN "ManufacturerName"
-F 5 "V10P45S-M3/86A" H 0   0   50  0001 C CNN "manufacturer-pn"
+F 5 "TPS2113A" H 0   0   50  0001 C CNN "manufacturer-pn"
 	1    6200 2750
 	0    1    1    0
@@
 F 3 "" H 2450 1100 50  0001 C CNN
 F 4 "Littelfuse" H 0   0   50  0001 C CNN "ManufacturerName"
-F 5 "2920L050DR" H 0   0   50  0001 C CNN "manufacturer-pn"
+F 5 " F8132CT-ND" H 0   0   50  0001 C CNN "manufacturer-pn"
 	1    2450 1100
 	0    1    1    0
@@
 F 0 "D4" H 3000 1650 50  0000 C CNN
 F 1 "D_Zener" H 3000 1450 50  0000 C CNN
-F 2 "Diodes_SMD:D_SOD-323_HandSoldering" H 3000 1550 50  0001 C CNN
+F 2 "Diodes_SMD:D_SMB_Handsoldering" H 3000 1550 50  0001 C CNN
 F 3 "" H 3000 1550 50  0000 C CNN
+F 4 "SMBJ5339B-TP" H 0   0   50  0001 C CNN "manufacturer-pn"
+F 5 "Micro Commercial Components (MCC)" H 0   0   50  0001 C CNN "ManufacturerName"
 	1    3000 1550
 	0    1    1    0
 $EndComp
-Text Notes 2300 1400 0    30   ~ 0
+Text Notes 2250 1400 0    30   ~ 0
 2920L050DR
 Text Label 10750 2750 2    60   ~ 0
@@
 F 2 "LEDs:LED_0603_HandSoldering" H 9850 4800 50  0001 C CNN
 F 3 "" H 9850 4800 50  0000 C CNN
+F 4 "Lite-On Inc." H 0   0   50  0001 C CNN "ManufacturerName"
+F 5 "LTST-C191KGKT" H 0   0   50  0001 C CNN "manufacturer-pn"
 	1    9850 4800
 	-1   0    0    1
@@
 F 3 "" H 4750 2600 50  0001 C CNN
 F 4 "Littelfuse" H 0   0   50  0001 C CNN "ManufacturerName"
-F 5 "2920L050DR" H 0   0   50  0001 C CNN "manufacturer-pn"
+F 5 " F8132CT-ND" H 0   0   50  0001 C CNN "manufacturer-pn"
 	1    4750 2600
 	0    1    1    0
@@
 F 0 "D5" H 5300 3150 50  0000 C CNN
 F 1 "D_Zener" H 5300 2950 50  0000 C CNN
-F 2 "Diodes_SMD:D_SOD-323_HandSoldering" H 5300 3050 50  0001 C CNN
+F 2 "Diodes_SMD:D_SMB_Handsoldering" H 5300 3050 50  0001 C CNN
 F 3 "" H 5300 3050 50  0000 C CNN
+F 4 "SMBJ5339B-TP" H 0   0   50  0001 C CNN "manufacturer-pn"
+F 5 "Micro Commercial Components (MCC)" H 0   0   50  0001 C CNN "ManufacturerName"
 	1    5300 3050
 	0    1    1    0
@@
 F 2 "LEDs:LED_0603_HandSoldering" H 5800 7250 50  0001 C CNN
 F 3 "~" H 5800 7250 50  0001 C CNN
+F 4 "Inolux" H 0   0   50  0001 C CNN "ManufacturerName"
+F 5 "IN-S63BTA " H 0   0   50  0001 C CNN "manufacturer-pn"
 	1    5800 7250
 	1    0    0    -1
@@
 F 2 "LEDs:LED_0603_HandSoldering" H 5800 5450 50  0001 C CNN
 F 3 "~" H 5800 5450 50  0001 C CNN
+F 4 "Inolux" H 0   0   50  0001 C CNN "ManufacturerName"
+F 5 "IN-S63BTA " H 0   0   50  0001 C CNN "manufacturer-pn"
 	1    5800 5450
 	1    0    0    -1

Commit message: fix some part typos
Parts:
- D8: ManufacturerName Vishay -> (none); manufacturer-pn TPS2113A -> (none)
- F1, F2: manufacturer-pn F8132CT-ND -> F8132CT-ND
- U5: ManufacturerName (none) -> Texas Instruments; manufacturer-pn (none) -> TPS2113A
Changed lines of the file:
@@
 F 2 "TO_SOT_Packages_SMD:TO-277A" H 6200 2750 50  0001 C CNN
 F 3 "" H 6200 2750 50  0000 C CNN
-F 4 "Vishay" H 0   0   50  0001 C CNN "ManufacturerName"
-F 5 "TPS2113A" H 0   0   50  0001 C CNN "manufacturer-pn"
+F 4 "" H 0   0   50  0001 C CNN "ManufacturerName"
+F 5 "" H 0   0   50  0001 C CNN "manufacturer-pn"
 	1    6200 2750
 	0    1    1    0
@@
 F 3 "" H 2450 1100 50  0001 C CNN
 F 4 "Littelfuse" H 0   0   50  0001 C CNN "ManufacturerName"
-F 5 " F8132CT-ND" H 0   0   50  0001 C CNN "manufacturer-pn"
+F 5 "F8132CT-ND" H 0   0   50  0001 C CNN "manufacturer-pn"
 	1    2450 1100
 	0    1    1    0
@@
 F 3 "" H 4750 2600 50  0001 C CNN
 F 4 "Littelfuse" H 0   0   50  0001 C CNN "ManufacturerName"
-F 5 " F8132CT-ND" H 0   0   50  0001 C CNN "manufacturer-pn"
+F 5 "F8132CT-ND" H 0   0   50  0001 C CNN "manufacturer-pn"
 	1    4750 2600
 	0    1    1    0
@@
 F 2 "Housings_SSOP:TSSOP-8_4.4x3mm_Pitch0.65mm" H 5950 1350 60  0001 C CNN
 F 3 "" H 5950 1350 60  0001 C CNN
+F 4 "Texas Instruments" H 0   0   50  0001 C CNN "ManufacturerName"
+F 5 "TPS2113A" H 0   0   50  0001 C CNN "manufacturer-pn"
 	1    5950 1350
 	1    0    0    -1

Commit message: someone set us up the BoM
Parts:
- D11, D7: manufacturer-pn IN-S63BTA -> IN-S63BTA
- D8: ManufacturerName (none) -> Vishay; manufacturer-pn (none) -> SS10PH10-M3/86A
- J12: ManufacturerName (none) -> Wurth; manufacturer-pn (none) -> 629105150521
- J13: ManufacturerName (none) -> Amphenol; manufacturer-pn (none) -> 12401610E4#2A
- Q5, Q6: ManufacturerName (none) -> Diodes Incorporated; manufacturer-pn (none) -> 2N7002-7-F
- R27, R28, R37, R38, R41, R42, R43: ManufacturerName (none) -> Panasonic Electronic Components; manufacturer-pn (none) -> ERA-3AEB104V
- R29, R30: ManufacturerName (none) -> Panasonic Electronic Components; manufacturer-pn (none) -> ERJ-PB3B5101V
- R33, R34: value NI -> 10K-NTC; ManufacturerName (none) -> Panasonic Electronic Components; manufacturer-pn (none) -> ERT-J1VG103JA
- R35: ManufacturerName (none) -> Panasonic Electronic Components; manufacturer-pn (none) -> ERJ-PB3B1001V
- R36: value NI -> 1K; ManufacturerName (none) -> Panasonic Electronic Components; manufacturer-pn (none) -> ERJ-PB3B1001V
- R39, R40: ManufacturerName (none) -> Panasonic Electronic Components; manufacturer-pn (none) -> ERA-3AEB331V
- TH1, TH2: value Thermistor_NTC -> NI
- U3, U4: ManufacturerName (none) -> Microchip Technology; manufacturer-pn (none) -> MCP73833T-AMI/UN
Changed lines of the file:
@@
 F 2 "Housings_SSOP:MSOP-10_3x3mm_Pitch0.5mm" H 2850 6300 60  0001 C CNN
 F 3 "" H 2850 6300 60  0001 C CNN
+F 4 "Microchip Technology" H 0   0   50  0001 C CNN "ManufacturerName"
+F 5 "MCP73833T-AMI/UN" H 0   0   50  0001 C CNN "manufacturer-pn"
 	1    2850 6300
 	1    0    0    -1
@@
 F 2 "Resistors_SMD:R_0603_HandSoldering" V 1680 6350 50  0001 C CNN
 F 3 "" H 1750 6350 50  0000 C CNN
+F 4 "Panasonic Electronic Components" H 0   0   50  0001 C CNN "ManufacturerName"
+F 5 "ERA-3AEB104V" H 0   0   50  0001 C CNN "manufacturer-pn"
 	1    1750 6350
 	0    1    1    0
@@
 F 2 "Resistors_SMD:R_0603_HandSoldering" V 3780 6750 50  0001 C CNN
 F 3 "" H 3850 6750 50  0000 C CNN
+F 4 "Panasonic Electronic Components" H 0   0   50  0001 C CNN "ManufacturerName"
+F 5 "ERJ-PB3B5101V" H 0   0   50  0001 C CNN "manufacturer-pn"
 	1    3850 6750
 	1    0    0    -1
@@
 AR Path="/5A6D4EDD/5AAD2FFD" Ref="R33"  Part="1"
 F 0 "R33" V 4330 6800 50  0000 C CNN
-F 1 "NI" V 4250 6800 50  0000 C CNN
+F 1 "10K-NTC" V 4250 6800 50  0000 C CNN
 F 2 "Resistors_SMD:R_0603_HandSoldering" V 4180 6800 50  0001 C CNN
 F 3 "" H 4250 6800 50  0000 C CNN
+F 4 "Panasonic Electronic Components" H 0   0   50  0001 C CNN "ManufacturerName"
+F 5 "ERT-J1VG103JA" H 0   0   50  0001 C CNN "manufacturer-pn"
 	1    4250 6800
 	1    0    0    -1
@@
 AR Path="/5A6D4EDD/5AAD3004" Ref="TH1"  Part="1"
 F 0 "TH1" V 4425 6800 50  0000 C CNN
-F 1 "Thermistor_NTC" V 4725 6800 50  0000 C CNN
+F 1 "NI" V 4725 6800 50  0000 C CNN
 F 2 "Capacitors_ThroughHole:CP_Radial_D4.0mm_P1.50mm" H 4600 6850 50  0001 C CNN
 F 3 "" H 4600 6850 50  0001 C CNN
@@
 F 2 "TO_SOT_Packages_SMD:TO-277A" H 6200 2750 50  0001 C CNN
 F 3 "" H 6200 2750 50  0000 C CNN
-F 4 "" H 0   0   50  0001 C CNN "ManufacturerName"
-F 5 "" H 0   0   50  0001 C CNN "manufacturer-pn"
+F 4 "Vishay" H 0   0   50  0001 C CNN "ManufacturerName"
+F 5 "SS10PH10-M3/86A " H 0   0   50  0001 C CNN "manufacturer-pn"
 	1    6200 2750
 	0    1    1    0
@@
 AR Path="/5A6D4EDD/5AB7020A" Ref="R36"  Part="1"
 F 0 "R36" V 10530 4800 50  0000 C CNN
-F 1 "NI" V 10450 4800 50  0000 C CNN
+F 1 "1K" V 10450 4800 50  0000 C CNN
 F 2 "Resistors_SMD:R_0603_HandSoldering" V 10380 4800 50  0001 C CNN
 F 3 "" H 10450 4800 50  0000 C CNN
+F 4 "Panasonic Electronic Components" H 0   0   50  0001 C CNN "ManufacturerName"
+F 5 "ERJ-PB3B1001V" H 0   0   50  0001 C CNN "manufacturer-pn"
 	1    10450 4800
 	0    -1   -1   0
@@
 F 2 "Connectors_USB:USB_Micro-B_Wuerth-629105150521_CircularHoles" H 1950 1450 50  0001 C CNN
 F 3 "" H 1950 1450 50  0001 C CNN
+F 4 "Wurth" H 0   0   50  0001 C CNN "ManufacturerName"
+F 5 "629105150521" H 0   0   50  0001 C CNN "manufacturer-pn"
 	1    1800 1500
 	-1   0    0    -1
@@
 F 2 "Connectors_USB:USB_C_Receptacle_Amphenol_12401610E4-2A_CircularHoles" H 3050 2700 50  0001 C CNN
 F 3 "" H 3050 2700 50  0001 C CNN
+F 4 "Amphenol" H 0   0   50  0001 C CNN "ManufacturerName"
+F 5 "12401610E4#2A" H 0   0   50  0001 C CNN "manufacturer-pn"
 	1    2900 2700
 	0    1    1    0
@@
 F 2 "Resistors_SMD:R_0603_HandSoldering" V 5080 1700 50  0001 C CNN
 F 3 "" H 5150 1700 50  0001 C CNN
+F 4 "Panasonic Electronic Components" H 0   0   50  0001 C CNN "ManufacturerName"
+F 5 "ERJ-PB3B1001V" H 0   0   50  0001 C CNN "manufacturer-pn"
 	1    5150 1700
 	1    0    0    -1
@@
 F 2 "TO_SOT_Packages_SMD:SOT-23W_Handsoldering" H 3950 7250 50  0001 C CNN
 F 3 "" H 3750 7150 50  0001 C CNN
+F 4 "Diodes Incorporated" H 0   0   50  0001 C CNN "ManufacturerName"
+F 5 "2N7002-7-F " H 0   0   50  0001 C CNN "manufacturer-pn"
 	1    3750 7150
 	1    0    0    -1
@@
 F 2 "Resistors_SMD:R_0603_HandSoldering" V 9930 3950 50  0001 C CNN
 F 3 "" H 10000 3950 50  0001 C CNN
+F 4 "Panasonic Electronic Components" H 0   0   50  0001 C CNN "ManufacturerName"
+F 5 "ERA-3AEB104V" H 0   0   50  0001 C CNN "manufacturer-pn"
 	1    10000 3950
 	0    -1   -1   0
@@
 F 2 "Resistors_SMD:R_0603_HandSoldering" V 4880 6850 50  0001 C CNN
 F 3 "" H 4950 6850 50  0001 C CNN
+F 4 "Panasonic Electronic Components" H 0   0   50  0001 C CNN "ManufacturerName"
+F 5 "ERA-3AEB104V" H 0   0   50  0001 C CNN "manufacturer-pn"
 	1    4950 6850
 	1    0    0    -1
@@
 F 2 "Resistors_SMD:R_0603_HandSoldering" V 6380 6200 50  0001 C CNN
 F 3 "" H 6450 6200 50  0001 C CNN
+F 4 "Panasonic Electronic Components" H 0   0   50  0001 C CNN "ManufacturerName"
+F 5 "ERA-3AEB104V" H 0   0   50  0001 C CNN "manufacturer-pn"
 	1    6450 6200
 	1    0    0    -1
@@
 F 2 "Resistors_SMD:R_0603_HandSoldering" V 5780 7050 50  0001 C CNN
 F 3 "" H 5850 7050 50  0001 C CNN
+F 4 "Panasonic Electronic Components" H 0   0   50  0001 C CNN "ManufacturerName"
+F 5 "ERA-3AEB331V" H 0   0   50  0001 C CNN "manufacturer-pn"
 	1    5850 7050
 	0    1    1    0
@@
 F 3 "~" H 5800 7250 50  0001 C CNN
 F 4 "Inolux" H 0   0   50  0001 C CNN "ManufacturerName"
-F 5 "IN-S63BTA " H 0   0   50  0001 C CNN "manufacturer-pn"
+F 5 "IN-S63BTA" H 0   0   50  0001 C CNN "manufacturer-pn"
 	1    5800 7250
 	1    0    0    -1
@@
 F 2 "Housings_SSOP:MSOP-10_3x3mm_Pitch0.5mm" H 2850 4500 60  0001 C CNN
 F 3 "" H 2850 4500 60  0001 C CNN
+F 4 "Microchip Technology" H 0   0   50  0001 C CNN "ManufacturerName"
+F 5 "MCP73833T-AMI/UN" H 0   0   50  0001 C CNN "manufacturer-pn"
 	1    2850 4500
 	1    0    0    -1
@@
 F 2 "Resistors_SMD:R_0603_HandSoldering" V 1680 4550 50  0001 C CNN
 F 3 "" H 1750 4550 50  0000 C CNN
+F 4 "Panasonic Electronic Components" H 0   0   50  0001 C CNN "ManufacturerName"
+F 5 "ERA-3AEB104V" H 0   0   50  0001 C CNN "manufacturer-pn"
 	1    1750 4550
 	0    1    1    0
@@
 F 2 "Resistors_SMD:R_0603_HandSoldering" V 3780 4950 50  0001 C CNN
 F 3 "" H 3850 4950 50  0000 C CNN
+F 4 "Panasonic Electronic Components" H 0   0   50  0001 C CNN "ManufacturerName"
+F 5 "ERJ-PB3B5101V" H 0   0   50  0001 C CNN "manufacturer-pn"
 	1    3850 4950
 	1    0    0    -1
@@
 AR Path="/5A6D4EDD/5C793D96" Ref="R34"  Part="1"
 F 0 "R34" V 4330 5000 50  0000 C CNN
-F 1 "NI" V 4250 5000 50  0000 C CNN
+F 1 "10K-NTC" V 4250 5000 50  0000 C CNN
 F 2 "Resistors_SMD:R_0603_HandSoldering" V 4180 5000 50  0001 C CNN
 F 3 "" H 4250 5000 50  0000 C CNN
+F 4 "Panasonic Electronic Components" H 0   0   50  0001 C CNN "ManufacturerName"
+F 5 "ERT-J1VG103JA" H 0   0   50  0001 C CNN "manufacturer-pn"
 	1    4250 5000
 	1    0    0    -1
@@
 AR Path="/5A6D4EDD/5C793D9D" Ref="TH2"  Part="1"
 F 0 "TH2" V 4425 5000 50  0000 C CNN
-F 1 "Thermistor_NTC" V 4725 5000 50  0000 C CNN
+F 1 "NI" V 4725 5000 50  0000 C CNN
 F 2 "Capacitors_ThroughHole:CP_Radial_D4.0mm_P1.50mm" H 4600 5050 50  0001 C CNN
 F 3 "" H 4600 5050 50  0001 C CNN
@@
 F 2 "TO_SOT_Packages_SMD:SOT-23W_Handsoldering" H 3950 5450 50  0001 C CNN
 F 3 "" H 3750 5350 50  0001 C CNN
+F 4 "Diodes Incorporated" H 0   0   50  0001 C CNN "ManufacturerName"
+F 5 "2N7002-7-F " H 0   0   50  0001 C CNN "manufacturer-pn"
 	1    3750 5350
 	1    0    0    -1
@@
 F 2 "Resistors_SMD:R_0603_HandSoldering" V 4880 5050 50  0001 C CNN
 F 3 "" H 4950 5050 50  0001 C CNN
+F 4 "Panasonic Electronic Components" H 0   0   50  0001 C CNN "ManufacturerName"
+F 5 "ERA-3AEB104V" H 0   0   50  0001 C CNN "manufacturer-pn"
 	1    4950 5050
 	1    0    0    -1
@@
 F 2 "Resistors_SMD:R_0603_HandSoldering" V 6380 4400 50  0001 C CNN
 F 3 "" H 6450 4400 50  0001 C CNN
+F 4 "Panasonic Electronic Components" H 0   0   50  0001 C CNN "ManufacturerName"
+F 5 "ERA-3AEB104V" H 0   0   50  0001 C CNN "manufacturer-pn"
 	1    6450 4400
 	1    0    0    -1
@@
 F 2 "Resistors_SMD:R_0603_HandSoldering" V 5780 5250 50  0001 C CNN
 F 3 "" H 5850 5250 50  0001 C CNN
+F 4 "Panasonic Electronic Components" H 0   0   50  0001 C CNN "ManufacturerName"
+F 5 "ERA-3AEB331V" H 0   0   50  0001 C CNN "manufacturer-pn"
 	1    5850 5250
 	0    1    1    0
@@
 F 3 "~" H 5800 5450 50  0001 C CNN
 F 4 "Inolux" H 0   0   50  0001 C CNN "ManufacturerName"
-F 5 "IN-S63BTA " H 0   0   50  0001 C CNN "manufacturer-pn"
+F 5 "IN-S63BTA" H 0   0   50  0001 C CNN "manufacturer-pn"
 	1    5800 5450
 	1    0    0    -1

Commit message: checked BoM
Parts:
- C39, C41: ManufacturerName TODO:C8 tantilum? Murata Electronics -> Murata Electronics
Changed lines of the file:
@@
 F 3 "" H 7350 2800 50  0000 C CNN
 F 4 "GRM21BD71A226ME44L" H 0   0   50  0001 C CNN "manufacturer-pn"
-F 5 "TODO:C8 tantilum? Murata Electronics" H 0   0   50  0001 C CNN "ManufacturerName"
+F 5 "Murata Electronics" H 0   0   50  0001 C CNN "ManufacturerName"
 	1    7350 2800
 	1    0    0    -1
@@
 F 3 "" H 8200 2800 50  0000 C CNN
 F 4 "GRM21BD71A226ME44L" H 0   0   50  0001 C CNN "manufacturer-pn"
-F 5 "TODO:C8 tantilum? Murata Electronics" H 0   0   50  0001 C CNN "ManufacturerName"
+F 5 "Murata Electronics" H 0   0   50  0001 C CNN "ManufacturerName"
 	1    8200 2800
 	1    0    0    -1

Commit message: eliminate old notes from schematic or move to notes.txt
Parts:
- F1, F2: manufacturer-pn F8132CT-ND -> 1812L050/60MR
Other:
- note removed: "1uF to 10uF should be fine; bigger is typically better,\n but we may get oscillation, need to test"
- note removed: "2920L050DR"
- note removed: "CMS1-12-R"
- note removed: "Consider thermal pad and SMD"
- note removed: "Keystone Electronics 1043"
- note removed: "MCP Datasheet typical: approx 5C-40C\nWith series resistor of 276 Ohm and parallel resistor of 149751 Ohm\n would give range of approx: 0C-45C"
- note removed: "REM3-0505S/A"
- note removed: "V10P45S-M3/86A"
Changed lines of the file:
@@
 	1    0    0    -1
 $EndComp
-Text Notes 9500 6000 0    30   ~ 0
-1uF to 10uF should be fine; bigger is typically better,\n but we may get oscillation, need to test
 $Comp
 L mcp73833:MCP73833 U3
@@
 	1    0    0    -1
 $EndComp
-Text Notes 2150 7400 0    30   ~ 0
-MCP Datasheet typical: approx 5C-40C\nWith series resistor of 276 Ohm and parallel resistor of 149751 Ohm\n would give range of approx: 0C-45C
 Text Label 11150 1150 2    60   ~ 0
 Bat2_Stat1
@@
 	1    0    0    -1
 $EndComp
-Text Notes 7650 3100 0    30   ~ 0
-CMS1-12-R
-Text Notes 6050 3000 1    30   ~ 0
-V10P45S-M3/86A
-Text Notes 9200 2600 0    30   ~ 0
-REM3-0505S/A
 Text Notes 6450 3350 0    30   ~ 0
 REM3-0505 Data sheet recommends\n1000uF through-hole Nippon Chemi-con KY series\nwe replaced with 3 SMD tantalums\n
@@
 F 3 "" H 2450 1100 50  0001 C CNN
 F 4 "Littelfuse" H 0   0   50  0001 C CNN "ManufacturerName"
-F 5 "F8132CT-ND" H 0   0   50  0001 C CNN "manufacturer-pn"
+F 5 "1812L050/60MR" H 0   0   50  0001 C CNN "manufacturer-pn"
 	1    2450 1100
 	0    1    1    0
@@
 	0    1    1    0
 $EndComp
-Text Notes 2250 1400 0    30   ~ 0
-2920L050DR
 Text Label 10750 2750 2    60   ~ 0
 V_ISO
@@
 F 3 "" H 4750 2600 50  0001 C CNN
 F 4 "Littelfuse" H 0   0   50  0001 C CNN "ManufacturerName"
-F 5 "F8132CT-ND" H 0   0   50  0001 C CNN "manufacturer-pn"
+F 5 "1812L050/60MR" H 0   0   50  0001 C CNN "manufacturer-pn"
 	1    4750 2600
 	0    1    1    0
@@
 	0    1    1    0
 $EndComp
-Text Notes 4600 2900 0    30   ~ 0
-2920L050DR
 $Comp
 L OpenHardwareHolterMonitor-rescue:GNDPWR #PWR022
@@
 	8500 2850 8550 2850
 Connection ~ 8500 2750
-Text Notes 6300 7400 0    30   ~ 0
-Keystone  Electronics 1043
 $Comp
 L Switch:SW_SPDT SW1
@@
 	1    0    0    -1
 $EndComp
-Text Notes 2150 5600 0    30   ~ 0
-MCP Datasheet typical: approx 5C-40C\nWith series resistor of 276 Ohm and parallel resistor of 149751 Ohm\n would give range of approx: 0C-45C
 Wire Wire Line
 	1600 4300 1750 4300
@@
 Wire Wire Line
 	1750 4300 1900 4300
-Text Notes 6300 5600 0    30   ~ 0
-Keystone  Electronics 1043
 $Comp
 L power:GND #PWR020
@@
 	1    0    0    -1
 $EndComp
-Text Notes 2150 5650 0    30   ~ 0
-Consider thermal pad and SMD
-Text Notes 2150 7450 0    30   ~ 0
-Consider thermal pad and SMD
 $Comp
 L OpenHardwareHolterMonitor-rescue:Q_PMOS_DGS-device Q11
