File: kicad-files/power.sch (KiCad schematic (older format))
At the start: 66 parts, among them J12 USB_OTG, J13 USB_C_Receptacle, Q10 Q_PMOS_DGS, Q11 Q_PMOS_DGS, Q5 Q_NMOS_DGS, Q6 Q_NMOS_DGS, Q7 Q_PMOS_DGS, Q8 Q_PMOS_DGS, Q9 Q_PMOS_DGS, SW1 SW_SPDT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

Commit message: fix schematic to use standard transistor pin numbers
Parts:
- Q10, Q11, Q7, Q8, Q9: value Q_PMOS_DGS -> DMG2305UX; symbol OpenHardwareHolterMonitor-rescue:Q_PMOS_DGS-device -> Device:Q_PMOS_GSD
- Q5, Q6: value Q_NMOS_DGS -> 2N7002; symbol OpenHardwareHolterMonitor-rescue:Q_NMOS_DGS-device -> Device:Q_NMOS_GSD
Connections:
- net Enable_Charging: now also Q5.1 (G), Q6.1 (G); no longer Q5.2 (G), Q6.2 (G)
- net GND: now also Q5.2 (S), Q6.2 (S); no longer Q5.3 (S), Q6.3 (S)
- net REGULATOR_IN: now also Q11.3 (D); no longer Q11.1 (D)
- net SWITCH_IN: now also Q11.2 (S); no longer Q11.3 (S)
- net at D6.2 (A), R42.1, U3.10 (VBAT)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: now also Q10.2 (S), Q8.2 (S); no longer Q10.3 (S), Q8.3 (S)
- net at BT1.1 (+), D14.2 (A), R40.1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: now also Q10.3 (D), Q8.1 (G); no longer Q10.1 (D), Q8.2 (G)
- net at R29.2: now also Q6.3 (D); no longer Q6.1 (D)
- net at SW1.2 (B): now also Q11.1 (G); no longer Q11.2 (G)
- net at D12.2 (A), R41.1, U4.10 (VBAT)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: now also Q7.2 (S), Q9.2 (S); no longer Q7.3 (S), Q9.3 (S)
- net at BT2.1 (+), D13.2 (A), R39.1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: now also Q7.1 (G), Q9.3 (D); no longer Q7.2 (G), Q9.1 (D)
- net at R30.2: now also Q5.3 (D); no longer Q5.1 (D)
- new net: Q10.1 (G), Q8.3 (D), R38.1
- new net: Q7.3 (D), Q9.1 (G), R37.1
Changed lines of the file:
@@
 Enable_Charging
 $Comp
-L OpenHardwareHolterMonitor-rescue:Q_NMOS_DGS-device Q6
+L Device:Q_NMOS_GSD Q6
 U 1 1 5BF1799C
 P 3750 7150
 F 0 "Q6" H 3955 7196 50  0000 L CNN
-F 1 "Q_NMOS_DGS" H 3955 7105 50  0000 L CNN
+F 1 "2N7002" H 3955 7105 50  0000 L CNN
 F 2 "TO_SOT_Packages_SMD:SOT-23W_Handsoldering" H 3950 7250 50  0001 C CNN
 F 3 "" H 3750 7150 50  0001 C CNN
@@
 	4250 7500 4600 7500
 $Comp
-L OpenHardwareHolterMonitor-rescue:Q_PMOS_DGS-device Q8
+L Device:Q_PMOS_GSD Q8
 U 1 1 5C337DE9
 P 5050 6200
 F 0 "Q8" H 5256 6154 50  0000 L CNN
-F 1 "Q_PMOS_DGS" H 5256 6245 50  0000 L CNN
+F 1 "DMG2305UX" H 5256 6245 50  0000 L CNN
 F 2 "TO_SOT_Packages_SMD:SOT-23_Handsoldering" H 5250 6300 50  0001 C CNN
 F 3 "" H 5050 6200 50  0001 C CNN
@@
 $EndComp
 $Comp
-L OpenHardwareHolterMonitor-rescue:Q_PMOS_DGS-device Q10
+L Device:Q_PMOS_GSD Q10
 U 1 1 5C34B9F0
 P 5650 6200
 F 0 "Q10" H 5856 6154 50  0000 L CNN
-F 1 "Q_PMOS_DGS" H 5856 6245 50  0000 L CNN
+F 1 "DMG2305UX" H 5856 6245 50  0000 L CNN
 F 2 "TO_SOT_Packages_SMD:SOT-23_Handsoldering" H 5850 6300 50  0001 C CNN
 F 3 "" H 5650 6200 50  0001 C CNN
@@
 $EndComp
 $Comp
-L OpenHardwareHolterMonitor-rescue:Q_NMOS_DGS-device Q5
+L Device:Q_NMOS_GSD Q5
 U 1 1 5C793DE1
 P 3750 5350
 F 0 "Q5" H 3955 5396 50  0000 L CNN
-F 1 "Q_NMOS_DGS" H 3955 5305 50  0000 L CNN
+F 1 "2N7002" H 3955 5305 50  0000 L CNN
 F 2 "TO_SOT_Packages_SMD:SOT-23W_Handsoldering" H 3950 5450 50  0001 C CNN
 F 3 "" H 3750 5350 50  0001 C CNN
@@
 	4250 5700 4600 5700
 $Comp
-L OpenHardwareHolterMonitor-rescue:Q_PMOS_DGS-device Q7
+L Device:Q_PMOS_GSD Q7
 U 1 1 5C793DF6
 P 5050 4400
 F 0 "Q7" H 5256 4354 50  0000 L CNN
-F 1 "Q_PMOS_DGS" H 5256 4445 50  0000 L CNN
+F 1 "DMG2305UX" H 5256 4445 50  0000 L CNN
 F 2 "TO_SOT_Packages_SMD:SOT-23_Handsoldering" H 5250 4500 50  0001 C CNN
 F 3 "" H 5050 4400 50  0001 C CNN
@@
 $EndComp
 $Comp
-L OpenHardwareHolterMonitor-rescue:Q_PMOS_DGS-device Q9
+L Device:Q_PMOS_GSD Q9
 U 1 1 5C793DFD
 P 5650 4400
 F 0 "Q9" H 5856 4354 50  0000 L CNN
-F 1 "Q_PMOS_DGS" H 5856 4445 50  0000 L CNN
+F 1 "DMG2305UX" H 5856 4445 50  0000 L CNN
 F 2 "TO_SOT_Packages_SMD:SOT-23_Handsoldering" H 5850 4500 50  0001 C CNN
 F 3 "" H 5650 4400 50  0001 C CNN
@@
 $EndComp
 $Comp
-L OpenHardwareHolterMonitor-rescue:Q_PMOS_DGS-device Q11
+L Device:Q_PMOS_GSD Q11
 U 1 1 5C48123F
 P 7700 4950
 F 0 "Q11" V 7906 4904 50  0000 L CNN
-F 1 "Q_PMOS_DGS" V 7550 4950 50  0000 L CNN
+F 1 "DMG2305UX" V 7550 4950 50  0000 L CNN
 F 2 "TO_SOT_Packages_SMD:SOT-23_Handsoldering" H 7900 5050 50  0001 C CNN
 F 3 "" H 7700 4950 50  0001 C CNN

Commit message: switch to consistent SOT-23 footprint
Parts:
- Q5, Q6: footprint TO_SOT_Packages_SMD:SOT-23W_Handsoldering -> TO_SOT_Packages_SMD:SOT-23_Handsoldering
Changed lines of the file:
@@
 F 0 "Q6" H 3955 7196 50  0000 L CNN
 F 1 "2N7002" H 3955 7105 50  0000 L CNN
-F 2 "TO_SOT_Packages_SMD:SOT-23W_Handsoldering" H 3950 7250 50  0001 C CNN
+F 2 "TO_SOT_Packages_SMD:SOT-23_Handsoldering" H 3950 7250 50  0001 C CNN
 F 3 "" H 3750 7150 50  0001 C CNN
 F 4 "Diodes Incorporated" H 0   0   50  0001 C CNN "ManufacturerName"
@@
 F 0 "Q5" H 3955 5396 50  0000 L CNN
 F 1 "2N7002" H 3955 5305 50  0000 L CNN
-F 2 "TO_SOT_Packages_SMD:SOT-23W_Handsoldering" H 3950 5450 50  0001 C CNN
+F 2 "TO_SOT_Packages_SMD:SOT-23_Handsoldering" H 3950 5450 50  0001 C CNN
 F 3 "" H 3750 5350 50  0001 C CNN
 F 4 "Diodes Incorporated" H 0   0   50  0001 C CNN "ManufacturerName"
